Commit message: Turned wheelchair 90 degrees to fix odometry errors.

File: wheelchair_description/urdf/wheelchair_with_swivels.xacro (robot description, xacro)
@@ -21,8 +21,21 @@
     <inertia ixx="${1/12 * weight * (3 * radius * radius + length * length)}" ixy="0" ixz="0" iyy="${1/12 * weight * (3 * radius*radius + length*length)}" iyz="0" izz="${1/2 * weight * radius*radius}" />
   </xacro:macro>
+  <link name="base_footprint">
+    <visual>
+      <origin xyz="0 0 0" rpy="0 0 0" />
+        <geometry>
+          <box size="0.001 0.001 0.001" />
+      </geometry>
+    </visual>
+  </link>
+  <joint name="base_footprint_joint" type="fixed">
+    <origin xyz=" 0 0 0" rpy="0 0 0"/>
+    <parent link="base_footprint"/>
+    <child link="base_link"/>
+  </joint>
   <link name="base_link">
     <visual>
       <geometry>
-        <box size="${chair_width} ${chair_length} ${chair_height}"/>
+        <box size="${chair_length} ${chair_width} ${chair_height}"/>
       </geometry>
       <material name="white">
@@ -32,5 +45,5 @@
     <collision>
       <geometry>
-        <box size="${chair_width} ${chair_length} ${chair_height}"/>
+        <box size="${chair_length} ${chair_width} ${chair_height}"/>
       </geometry>
     </collision>
@@ -44,5 +57,5 @@
     <visual>
       <geometry>
-        <box size="${legs_width} ${legs_length} ${legs_height}"/>
+        <box size="${legs_length} ${legs_width} ${legs_height}"/>
       </geometry>
       <material name="white">
@@ -52,5 +65,5 @@
     <collision>
       <geometry>
-        <box size="${legs_width} ${legs_length} ${legs_height}"/>
+        <box size="${legs_length} ${legs_width} ${legs_height}"/>
       </geometry>
     </collision>
@@ -64,5 +77,5 @@
     <parent link="base_link"/>
     <child link="legs"/>
-    <origin rpy="0 0 0" xyz="0 -${chair_length/2 + 0.4064/2} -${chair_height/2 - 0.4064/2}"/> <!--chair_height/4 + chair_height/8 because this is relative to the center of the bar -->
+    <origin rpy="0 0 0" xyz="${chair_length/2 + 0.4064/2} 0 -${chair_height/2 - 0.4064/2}"/> <!--chair_height/4 + chair_height/8 because this is relative to the center of the bar -->
   </joint>
 <!--Right Bar -->
@@ -70,5 +83,5 @@
     <visual>
       <geometry>
-        <box size="${chair_width/4} ${chair_length + chair_length/4} ${chair_height/8}"/>
+        <box size="${chair_length + chair_length/4} ${chair_width/4} ${chair_height/8}"/>
       </geometry>
       <material name="white">
@@ -78,5 +91,5 @@
     <collision>
       <geometry>
-        <box size="${chair_width/4} ${chair_length} ${chair_height/8}"/>
+        <box size="${chair_length + chair_length/4} ${chair_width/4} ${chair_height/8}"/>
       </geometry>
     </collision>
@@ -90,5 +103,5 @@
     <parent link="base_link"/>
     <child link="right_bar"/>
-    <origin rpy="0 0 0" xyz="${chair_width/2} 0.0 -${chair_height/4 + chair_height/8}"/> <!--chair_height/4 + chair_height/8 because this is relative to the center of the bar -->
+    <origin rpy="0 0 0" xyz="0.0 ${chair_width/2} -${chair_height/4 + chair_height/8}"/> <!--chair_height/4 + chair_height/8 because this is relative to the center of the bar -->
   </joint>
 <!--Left Bar -->
@@ -96,5 +109,5 @@
     <visual>
       <geometry>
-        <box size="${chair_width/4} ${chair_length + chair_length/4} ${chair_height/8}"/>
+        <box size="${chair_length + chair_length/4} ${chair_width/4} ${chair_height/8}"/>
       </geometry>
       <material name="white">
@@ -104,5 +117,5 @@
     <collision>
       <geometry>
-        <box size="${chair_width/4} ${chair_length} ${chair_height/8}"/>
+        <box size="${chair_length + chair_length/4} ${chair_width/4} ${chair_height/8}"/>
       </geometry>
     </collision>
@@ -116,12 +129,12 @@
     <parent link="base_link"/>
     <child link="left_bar"/>
-    <origin rpy="0 0 0" xyz="-${chair_width/2} 0.0 -${chair_height/4 + chair_height/8}"/> <!--chair_height/4 + chair_height/8 because this is relative to the center of the bar -->
+    <origin rpy="0 0 0" xyz="0.0 -${chair_width/2} -${chair_height/4 + chair_height/8}"/> <!--chair_height/4 + chair_height/8 because this is relative to the center of the bar -->
   </joint>
 <!--Main Wheels -->
   <joint name="right_main_wheel_joint" type="continuous">
-    <axis xyz="0 0 1"/>
+    <axis xyz="0 0 -1"/>
     <parent link="right_bar"/>
     <child link="right_main_wheel"/>
-    <origin rpy="0 1.57075 0" xyz="0.0 0.0 -${chair_height/8-0.076}"/>
+    <origin rpy="1.57075 0 0" xyz="0.0 0.0 -${chair_height/8-0.076}"/>
   </joint>
   <link name="right_main_wheel">
@@ -145,8 +158,8 @@
   </link>
   <joint name="left_main_wheel_joint" type="continuous">
-    <axis xyz="0 0 1"/>
+    <axis xyz="0 0 -1"/>
     <parent link="left_bar"/>
     <child link="left_main_wheel"/>
-    <origin rpy="0 1.57075 0" xyz="0.0 0.0 -${chair_height/8-0.076}"/>
+    <origin rpy="1.57075 0 0" xyz="0.0 0.0 -${chair_height/8-0.076}"/>
   </joint>
   <link name="left_main_wheel">
@@ -178,5 +191,4 @@
     </visual>
     <collision>
-      <origin xyz="0.0 0 0" rpy="0 0 0"/>
       <geometry>
         <box size="0.05 0.05 0.1"/>
@@ -190,5 +202,5 @@
   <joint name="right_scanner_joint" type="fixed">
     <axis xyz="0 0 0" />
-    <origin xyz="${0.05/2} -${chair_length/2 - 0.05/2 + chair_length/8} ${chair_height/16 + 0.05}" rpy="0 0 0"/>
+    <origin xyz="${chair_length/2 - 0.05/2 + chair_length/8} -${0.05/2} ${chair_height/16 + 0.05}" rpy="0 0 0"/>
     <parent link="right_bar"/>
     <child link="right_scanner"/>
@@ -213,5 +225,5 @@
   <joint name="left_scanner_joint" type="fixed">
     <axis xyz="0 0 0" />
-    <origin xyz="-${0.05/2} -${chair_length/2 - 0.05/2 + chair_length/8} ${chair_height/16 + 0.05}" rpy="0 0 -3.14"/>
+    <origin xyz="${chair_length/2 - 0.05/2 + chair_length/8} -${0.05/2} ${chair_height/16 + 0.05}" rpy="0 0 -3.14159265359"/>
     <parent link="left_bar"/>
     <child link="left_scanner"/>
@@ -241,5 +253,5 @@
     <parent link="right_bar"/>
     <child link="front_right_swivel"/>
-    <origin rpy="0 0 0" xyz="0.0 -${chair_length/2} -${chair_height/8}"/>
+    <origin rpy="0 0 0" xyz="-${chair_length/2} 0.0 -${chair_height/8}"/>
     <dynamics damping="0.0" friction="0.5" />
   </joint>
@@ -248,5 +260,5 @@
     <parent link="front_right_swivel"/>
     <child link="front_right_wheel"/>
-    <origin rpy="0 1.57075 0" xyz="0 0.065 0"/>
+    <origin rpy="1.57075 0 0" xyz="0.065 0 0"/>
     <dynamics damping="1.0" friction="1.5" />
   </joint>
@@ -267,6 +279,6 @@
         <friction>
           <ode>
-            <mu>100.0</mu>
-            <mu2>100.0</mu2>
+            <mu>1.0</mu>
+            <mu2>1.0</mu2>
           </ode>
         </friction>
@@ -301,5 +313,5 @@
     <parent link="left_bar"/>
     <child link="front_left_swivel"/>
-    <origin rpy="0 0 0" xyz="0.0 -${chair_length/2} -${chair_height/8}"/>
+    <origin rpy="0 0 0" xyz="-${chair_length/2} 0.0 -${chair_height/8}"/>
     <dynamics damping="0.0" friction="0.5" />
   </joint>
@@ -308,5 +320,5 @@
     <parent link="front_left_swivel"/>
     <child link="front_left_wheel"/>
-    <origin rpy="0 1.57075 0" xyz="0 0.065 0"/>
+    <origin rpy="1.57075 0 0" xyz="0.065 0 0"/>
     <dynamics damping="0" friction="0.5" />
   </joint>
@@ -327,6 +339,6 @@
         <friction>
           <ode>
-            <mu>100.0</mu>
-            <mu2>100.0</mu2>
+            <mu>1.0</mu>
+            <mu2>1.0</mu2>
           </ode>
         </friction>
@@ -362,5 +374,5 @@
     <parent link="right_bar"/>
     <child link="rear_right_swivel"/>
-    <origin rpy="0 0 0" xyz="0.0 ${chair_length/2} -${chair_height/8}"/>
+    <origin rpy="0 0 0" xyz="${chair_length/2} 0.0 -${chair_height/8}"/>
     <dynamics damping="0.0" friction="0.5" />
   </joint>
@@ -369,5 +381,5 @@
     <parent link="rear_right_swivel"/>
     <child link="rear_right_wheel"/>
-    <origin rpy="0 1.57075 0" xyz="0 0.065 0"/>
+    <origin rpy="1.57075 0 0" xyz="0.065 0 0"/>
     <dynamics damping="0" friction="0.5" />
   </joint>
@@ -388,6 +400,6 @@
         <friction>
           <ode>
-            <mu>100.0</mu>
-            <mu2>100.0</mu2>
+            <mu>1.0</mu>
+            <mu2>1.0</mu2>
           </ode>
         </friction>
@@ -422,5 +434,5 @@
     <parent link="left_bar"/>
     <child link="rear_left_swivel"/>
-    <origin rpy="0 0 0" xyz="0.0 ${chair_length/2} -${chair_height/8}"/>
+    <origin rpy="0 0 0" xyz="${chair_length/2} 0.0 -${chair_height/8}"/>
     <dynamics damping="0.0" friction="0.5" />
   </joint>
@@ -429,5 +441,5 @@
     <parent link="rear_left_swivel"/>
     <child link="rear_left_wheel"/>
-    <origin rpy="0 1.57075 0" xyz="0 0.065 0"/>
+    <origin rpy="1.57075 0 0" xyz="0.065 0 0"/>
     <dynamics damping="0" friction="0.5" />
   </joint>
@@ -448,6 +460,6 @@
         <friction>
           <ode>
-            <mu>100.0</mu>
-            <mu2>100.0</mu2>
+            <mu>1.0</mu>
+            <mu2>1.0</mu2>
           </ode>
         </friction>
@@ -463,8 +475,8 @@
     <alwaysOn>true</alwaysOn>
     <updateRate>50</updateRate>
-    <leftJoint>right_main_wheel_joint</leftJoint>
-    <rightJoint>left_main_wheel_joint</rightJoint>
-    <wheelSeparation>0.5380</wheelSeparation>
-    <wheelDiameter>${main_wheel_radius}</wheelDiameter>
+    <leftJoint>left_main_wheel_joint</leftJoint>
+    <rightJoint>right_main_wheel_joint</rightJoint>
+    <wheelSeparation>${chair_width}</wheelSeparation>
+    <wheelDiameter>${main_wheel_radius*2}</wheelDiameter>
     <torque>20</torque>
     <commandTopic>cmd_vel</commandTopic>
@@ -484,6 +496,6 @@
             <samples>720</samples>
             <resolution>1</resolution>
-            <min_angle>-2.35619449</min_angle>
-            <max_angle>2.35619449</max_angle>
+            <min_angle>0</min_angle>
+            <max_angle>3.14159265359</max_angle>
           </horizontal>
         </scan>
@@ -495,8 +507,4 @@
         <noise>
           <type>gaussian</type>
-          <!-- Noise parameters based on published spec for Hokuyo laser
-               achieving "+-30mm" accuracy at range < 10m.  A mean of 0.0m and
-               stddev of 0.01m will put 99.7% of samples within 0.03m of the true
-               reading. -->
           <mean>0.0</mean>
           <stddev>0.01</stddev>
@@ -504,5 +512,5 @@
       </ray>
       <plugin name="gazebo_ros_head_hokuyo_controller" filename="libgazebo_ros_gpu_laser.so">
-        <topicName>/wheelchair/laser/scan</topicName>
+        <topicName>/wheelchair_lasers/right</topicName>
         <frameName>right_scanner</frameName>
       </plugin>
@@ -512,5 +520,5 @@
     <sensor type="gpu_ray" name="head_hokuyo_sensor2">
       <pose>0 0 0 0 0 0</pose>
-      <visualize>false</visualize>
+      <visualize>true</visualize>
       <update_rate>40</update_rate>
       <ray>
@@ -519,6 +527,6 @@
             <samples>720</samples>
             <resolution>1</resolution>
-            <min_angle>-2.35619449</min_angle>
-            <max_angle>2.35619449</max_angle>
+            <min_angle>0</min_angle>
+            <max_angle>3.14159265359</max_angle>
           </horizontal>
         </scan>
@@ -535,5 +543,5 @@
       </ray>
       <plugin name="gazebo_ros_head_hokuyo_controller2" filename="libgazebo_ros_gpu_laser.so">
-        <topicName>/wheelchair/laser2/scan</topicName>
+        <topicName>/wheelchair_lasers/left</topicName>
         <frameName>left_scanner</frameName>
       </plugin>
