Commit message: Needed to rotate wheelchair 90 degrees...
NOTE: THIS MAY BREAK SIMULATION -- CHECK BACK HERE LATER.

File: wheelchair_description/urdf/wheelchair.xacro (robot description, xacro)
@@ -12,5 +12,5 @@
   <xacro:property name="main_wheel_radius" value=".165" />
   <xacro:property name="main_wheel_weight" value="2.0" />
-  <xacro:property name="small_wheel_radius" value=".0885" />
+  <xacro:property name="small_wheel_radius" value=".089" />
   <xacro:property name="small_wheel_length" value=".05" />
   <xacro:property name="small_wheel_weight" value="1.0" />
@@ -21,8 +21,21 @@
     <inertia ixx="${1/12 * weight * (3 * radius * radius + length * length)}" ixy="0" ixz="0" iyy="${1/12 * weight * (3 * radius*radius + length*length)}" iyz="0" izz="${1/2 * weight * radius*radius}" />
   </xacro:macro>
+  <link name="base_footprint">
+    <visual>
+      <origin xyz="0 0 0" rpy="0 0 0" />
+        <geometry>
+          <box size="0.001 0.001 0.001" />
+      </geometry>
+    </visual>
+  </link>
+  <joint name="base_footprint_joint" type="fixed">
+    <origin xyz=" 0 0 0.7" rpy="0 0 0"/>
+    <parent link="base_footprint"/>
+    <child link="base_link"/>
+  </joint>
   <link name="base_link">
     <visual>
       <geometry>
-        <box size="${chair_width} ${chair_length} ${chair_height}"/>
+        <box size="${chair_length} ${chair_width} ${chair_height}"/>
       </geometry>
       <material name="white">
@@ -32,5 +45,5 @@
     <collision>
       <geometry>
-        <box size="${chair_width} ${chair_length} ${chair_height}"/>
+        <box size="${chair_length} ${chair_width} ${chair_height}"/>
       </geometry>
     </collision>
@@ -44,5 +57,5 @@
     <visual>
       <geometry>
-        <box size="${legs_width} ${legs_length} ${legs_height}"/>
+        <box size="${legs_length} ${legs_width} ${legs_height}"/>
       </geometry>
       <material name="white">
@@ -52,5 +65,5 @@
     <collision>
       <geometry>
-        <box size="${legs_width} ${legs_length} ${legs_height}"/>
+        <box size="${legs_length} ${legs_width} ${legs_height}"/>
       </geometry>
     </collision>
@@ -64,5 +77,5 @@
     <parent link="base_link"/>
     <child link="legs"/>
-    <origin rpy="0 0 0" xyz="0 -${chair_length/2 + 0.4064/2} -${chair_height/2 - 0.4064/2}"/> <!--chair_height/4 + chair_height/8 because this is relative to the center of the bar -->
+    <origin rpy="0 0 0" xyz="${chair_length/2 + 0.4064/2} 0 -${chair_height/2 - 0.4064/2}"/> <!--chair_height/4 + chair_height/8 because this is relative to the center of the bar -->
   </joint>
 <!--Right Bar -->
@@ -70,5 +83,5 @@
     <visual>
       <geometry>
-        <box size="${chair_width/4} ${chair_length + chair_length/4} ${chair_height/8}"/>
+        <box size="${chair_length + chair_length/4} ${chair_width/4} ${chair_height/8}"/>
       </geometry>
       <material name="white">
@@ -78,5 +91,5 @@
     <collision>
       <geometry>
-        <box size="${chair_width/4} ${chair_length} ${chair_height/8}"/>
+        <box size="${chair_length + chair_length/4} ${chair_width/4} ${chair_height/8}"/>
       </geometry>
     </collision>
@@ -90,5 +103,5 @@
     <parent link="base_link"/>
     <child link="right_bar"/>
-    <origin rpy="0 0 0" xyz="${chair_width/2} 0.0 -${chair_height/4 + chair_height/8}"/> <!--chair_height/4 + chair_height/8 because this is relative to the center of the bar -->
+    <origin rpy="0 0 0" xyz="0.0 ${chair_width/2} -${chair_height/4 + chair_height/8}"/> <!--chair_height/4 + chair_height/8 because this is relative to the center of the bar -->
   </joint>
 <!--Left Bar -->
@@ -96,5 +109,5 @@
     <visual>
       <geometry>
-        <box size="${chair_width/4} ${chair_length + chair_length/4} ${chair_height/8}"/>
+        <box size="${chair_length + chair_length/4} ${chair_width/4} ${chair_height/8}"/>
       </geometry>
       <material name="white">
@@ -104,5 +117,5 @@
     <collision>
       <geometry>
-        <box size="${chair_width/4} ${chair_length} ${chair_height/8}"/>
+        <box size="${chair_length + chair_length/4} ${chair_width/4} ${chair_height/8}"/>
       </geometry>
     </collision>
@@ -116,12 +129,12 @@
     <parent link="base_link"/>
     <child link="left_bar"/>
-    <origin rpy="0 0 0" xyz="-${chair_width/2} 0.0 -${chair_height/4 + chair_height/8}"/> <!--chair_height/4 + chair_height/8 because this is relative to the center of the bar -->
+    <origin rpy="0 0 0" xyz="0.0 -${chair_width/2} -${chair_height/4 + chair_height/8}"/> <!--chair_height/4 + chair_height/8 because this is relative to the center of the bar -->
   </joint>
 <!--Main Wheels -->
   <joint name="right_main_wheel_joint" type="continuous">
-    <axis xyz="0 0 1"/>
+    <axis xyz="0 0 -1"/>
     <parent link="right_bar"/>
     <child link="right_main_wheel"/>
-    <origin rpy="0 1.57075 0" xyz="0.0 0.0 -${chair_height/8-0.076}"/>
+    <origin rpy="1.57075 0 0" xyz="0.0 0.0 -${chair_height/8-0.076}"/>
   </joint>
   <link name="right_main_wheel">
@@ -145,8 +158,8 @@
   </link>
   <joint name="left_main_wheel_joint" type="continuous">
-    <axis xyz="0 0 1"/>
+    <axis xyz="0 0 -1"/>
     <parent link="left_bar"/>
     <child link="left_main_wheel"/>
-    <origin rpy="0 1.57075 0" xyz="0.0 0.0 -${chair_height/8-0.076}"/>
+    <origin rpy="1.57075 0 0" xyz="0.0 0.0 -${chair_height/8-0.076}"/>
   </joint>
   <link name="left_main_wheel">
@@ -178,7 +191,6 @@
     </visual>
     <collision>
-      <origin xyz="0.0 0 0" rpy="0 0 0"/>
-      <geometry>
-        <box size="0.1 0.1 0.1"/>
+      <geometry>
+        <box size="0.05 0.05 0.1"/>
       </geometry>
     </collision>
@@ -190,5 +202,5 @@
   <joint name="right_scanner_joint" type="fixed">
     <axis xyz="0 0 0" />
-    <origin xyz="${0.05/2} -${chair_length/2 - 0.05/2 + chair_length/8} ${chair_height/16 + 0.05}" rpy="0 0 0"/>
+    <origin xyz="${chair_length/2 - 0.05/2 + chair_length/8} -${0.05/2} ${chair_height/16 + 0.05}" rpy="0 0 1.5707"/>
     <parent link="right_bar"/>
     <child link="right_scanner"/>
@@ -203,5 +215,5 @@
     <collision>
       <geometry>
-        <box size="0.1 0.1 0.1"/>
+        <box size="0.05 0.05 0.1"/>
       </geometry>
     </collision>
@@ -213,15 +225,41 @@
   <joint name="left_scanner_joint" type="fixed">
     <axis xyz="0 0 0" />
-    <origin xyz="-${0.05/2} -${chair_length/2 - 0.05/2 + chair_length/8} ${chair_height/16 + 0.05}" rpy="0 0 -3.14"/>
+    <origin xyz="${chair_length/2 - 0.05/2 + chair_length/8} -${0.05/2} ${chair_height/16 + 0.05}" rpy="0 0 -1.5707"/>
     <parent link="left_bar"/>
     <child link="left_scanner"/>
   </joint>
 <!--Front Wheels -->
+  <link name="front_right_swivel">
+    <visual>
+      <geometry>
+        <cylinder length="0.065" radius="0.01"/>
+      </geometry>
+      <material name="white">
+        <color rgba="0 0 0 1"/>
+      </material>
+    </visual>
+    <collision>
+      <geometry>
+        <cylinder length="0.065" radius="0.01"/>
+      </geometry>
+    </collision>
+    <inertial>
+      <mass value=".1"/>
+      <xacro:cylinder_intertia length="0.065" radius="0.01" weight="0.1" />
+    </inertial>
+  </link>
+   <joint name="front_right_swivel_joint" type="continuous">
+    <axis xyz="0 0 1"/>
+    <parent link="right_bar"/>
+    <child link="front_right_swivel"/>
+    <origin rpy="0 0 0" xyz="-${chair_length/2} 0.0 -${chair_height/8}"/>
+    <dynamics damping="0.0" friction="0.5" />
+  </joint>
   <joint name="front_right_wheel_joint" type="continuous">
     <axis xyz="0 0 1"/>
-    <parent link="right_bar"/>
+    <parent link="front_right_swivel"/>
     <child link="front_right_wheel"/>
-    <origin rpy="0 1.57075 0" xyz="0.0 ${chair_length/2} -${chair_height/8}"/>
-    <dynamics damping="0.0" friction="0.5" />
+    <origin rpy="1.57075 0 0" xyz="0.065 0 0"/>
+    <dynamics damping="1.0" friction="1.5" />
   </joint>
   <link name="front_right_wheel">
@@ -238,4 +276,12 @@
         <cylinder length="${small_wheel_length}" radius="${small_wheel_radius}"/>
       </geometry>
+      <surface>
+        <friction>
+          <ode>
+            <mu>1.0</mu>
+            <mu2>1.0</mu2>
+          </ode>
+        </friction>
+      </surface>
     </collision>
     <inertial>
@@ -244,10 +290,36 @@
     </inertial>
   </link>
-<joint name="front_left_wheel_joint" type="continuous">
+  <link name="front_left_swivel">
+    <visual>
+      <geometry>
+        <cylinder length="0.065" radius="0.01"/>
+      </geometry>
+      <material name="white">
+        <color rgba="0 0 0 1"/>
+      </material>
+    </visual>
+    <collision>
+      <geometry>
+        <cylinder length="0.065" radius="0.01"/>
+      </geometry>
+    </collision>
+    <inertial>
+      <mass value=".1"/>
+      <xacro:cylinder_intertia length="0.065" radius="0.01" weight="0.1" />
+    </inertial>
+  </link>
+   <joint name="front_left_swivel_joint" type="continuous">
     <axis xyz="0 0 1"/>
     <parent link="left_bar"/>
+    <child link="front_left_swivel"/>
+    <origin rpy="0 0 0" xyz="-${chair_length/2} 0.0 -${chair_height/8}"/>
+    <dynamics damping="0.0" friction="0.5" />
+  </joint>
+  <joint name="front_left_wheel_joint" type="continuous">
+    <axis xyz="0 0 1"/>
+    <parent link="front_left_swivel"/>
     <child link="front_left_wheel"/>
-    <origin rpy="0 1.57075 0" xyz="0.0 ${chair_length/2} -${chair_height/8}"/>
-    <dynamics damping="0.0" friction="0.5" />
+    <origin rpy="1.57075 0 0" xyz="0.065 0 0"/>
+    <dynamics damping="0" friction="0.5" />
   </joint>
   <link name="front_left_wheel">
@@ -264,4 +336,12 @@
         <cylinder length="0.05" radius="${small_wheel_radius}"/>
       </geometry>
+      <surface>
+        <friction>
+          <ode>
+            <mu>1.0</mu>
+            <mu2>1.0</mu2>
+          </ode>
+        </friction>
+      </surface>
     </collision>
     <inertial>
@@ -271,9 +351,36 @@
   </link>
 <!--Rear Wheels -->
+  <link name="rear_right_swivel">
+    <visual>
+      <geometry>
+        <cylinder length="0.065" radius="0.01"/>
+      </geometry>
+      <material name="white">
+        <color rgba="0 0 0 1"/>
+      </material>
+    </visual>
+    <collision>
+      <geometry>
+        <cylinder length="0.065" radius="0.01"/>
+      </geometry>
+    </collision>
+    <inertial>
+      <mass value=".1"/>
+      <xacro:cylinder_intertia length="0.065" radius="0.01" weight="0.1" />
+    </inertial>
+  </link>
+   <joint name="rear_right_swivel_joint" type="continuous">
+    <axis xyz="0 0 1"/>
+    <parent link="right_bar"/>
+    <child link="rear_right_swivel"/>
+    <origin rpy="0 0 0" xyz="${chair_length/2} 0.0 -${chair_height/8}"/>
+    <dynamics damping="0.0" friction="0.5" />
+  </joint>
   <joint name="rear_right_wheel_joint" type="continuous">
     <axis xyz="0 0 1"/>
-    <parent link="right_bar"/>
+    <parent link="rear_right_swivel"/>
     <child link="rear_right_wheel"/>
-    <origin rpy="0 1.57075 0" xyz="0.0 -${chair_length/2} -${chair_height/8}"/>
+    <origin rpy="1.57075 0 0" xyz="0.065 0 0"/>
+    <dynamics damping="0" friction="0.5" />
   </joint>
   <link name="rear_right_wheel">
@@ -290,4 +397,12 @@
         <cylinder length="0.05" radius="${small_wheel_radius}"/>
       </geometry>
+      <surface>
+        <friction>
+          <ode>
+            <mu>1.0</mu>
+            <mu2>1.0</mu2>
+          </ode>
+        </friction>
+      </surface>
     </collision>
     <inertial>
@@ -296,9 +411,36 @@
     </inertial>
   </link>
+  <link name="rear_left_swivel">
+    <visual>
+      <geometry>
+        <cylinder length="0.065" radius="0.01"/>
+      </geometry>
+      <material name="white">
+        <color rgba="0 0 0 1"/>
+      </material>
+    </visual>
+    <collision>
+      <geometry>
+        <cylinder length="0.065" radius="0.01"/>
+      </geometry>
+    </collision>
+    <inertial>
+      <mass value=".1"/>
+      <xacro:cylinder_intertia length="0.065" radius="0.01" weight="0.1" />
+    </inertial>
+  </link>
+   <joint name="rear_left_swivel_joint" type="continuous">
+    <axis xyz="0 0 1"/>
+    <parent link="left_bar"/>
+    <child link="rear_left_swivel"/>
+    <origin rpy="0 0 0" xyz="${chair_length/2} 0.0 -${chair_height/8}"/>
+    <dynamics damping="0.0" friction="0.5" />
+  </joint>
   <joint name="rear_left_wheel_joint" type="continuous">
     <axis xyz="0 0 1"/>
-    <parent link="left_bar"/>
+    <parent link="rear_left_swivel"/>
     <child link="rear_left_wheel"/>
-    <origin rpy="0 1.57075 0" xyz="0.0 -${chair_length/2} -${chair_height/8}"/>
+    <origin rpy="1.57075 0 0" xyz="0.065 0 0"/>
+    <dynamics damping="0" friction="0.5" />
   </joint>
   <link name="rear_left_wheel">
@@ -315,4 +457,12 @@
         <cylinder length="0.05" radius="${small_wheel_radius}"/>
       </geometry>
+      <surface>
+        <friction>
+          <ode>
+            <mu>1.0</mu>
+            <mu2>1.0</mu2>
+          </ode>
+        </friction>
+      </surface>
     </collision>
     <inertial>
@@ -321,316 +471,3 @@
     </inertial>
   </link>
-<gazebo>
-  <plugin name="differential_drive_controller" filename="libgazebo_ros_diff_drive.so">
-    <alwaysOn>true</alwaysOn>
-    <updateRate>50</updateRate>
-    <leftJoint>right_main_wheel_joint</leftJoint>
-    <rightJoint>left_main_wheel_joint</rightJoint>
-    <wheelSeparation>0.5380</wheelSeparation>
-    <wheelDiameter>${main_wheel_radius}</wheelDiameter>
-    <torque>20</torque>
-    <commandTopic>cmd_vel</commandTopic>
-    <odometryTopic>odom</odometryTopic>
-    <odometryFrame>odom</odometryFrame>
-    <robotBaseFrame>base_footprint</robotBaseFrame>
-  </plugin>
-</gazebo>
-<gazebo reference="right_scanner">
-    <sensor type="gpu_ray" name="head_hokuyo_sensor">
-      <pose>0 0 0 0 0 0</pose>
-      <visualize>true</visualize>
-      <update_rate>40</update_rate>
-      <ray>
-        <scan>
-          <horizontal>
-            <samples>720</samples>
-            <resolution>1</resolution>
-            <min_angle>-2.35619449</min_angle>
-            <max_angle>2.35619449</max_angle>
-          </horizontal>
-        </scan>
-        <range>
-          <min>0.10</min>
-          <max>30.0</max>
-          <resolution>0.01</resolution>
-        </range>
-        <noise>
-          <type>gaussian</type>
-          <!-- Noise parameters based on published spec for Hokuyo laser
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