Commit message: Added c300 wheelchair and fixed a friction bug in the original wheelchair.

File: wheelchair_description/urdf/wheelchair_description_c300.xacro (robot description, xacro)
@@ -155,5 +155,5 @@
     <parent link="right_bar"/>
     <child link="right_main_wheel"/>
-    <origin rpy="1.57075 0 0" xyz="0.0 0.0 -${chair_height/8-0.076}"/>
+    <origin rpy="1.57075 0 0" xyz="0.2 0.0 -${chair_height/8-0.076}"/>
   </joint>
   <link name="right_main_wheel">
@@ -180,5 +180,5 @@
     <parent link="left_bar"/>
     <child link="left_main_wheel"/>
-    <origin rpy="1.57075 0 0" xyz="0.0 0.0 -${chair_height/8-0.076}"/>
+    <origin rpy="1.57075 0 0" xyz="0.2 0.0 -${chair_height/8-0.076}"/>
   </joint>
   <link name="left_main_wheel">
@@ -280,5 +280,5 @@
     <child link="front_right_wheel"/>
     <origin rpy="1.57075 0 0" xyz="0.065 0 0"/>
-    <dynamics damping="0.0" friction="0.5" />
+    <dynamics damping="0" friction="0.5" />
   </joint>
   <link name="front_right_wheel">
@@ -370,123 +370,3 @@
   </link>
 <!--Rear Wheels -->
-  <link name="rear_right_swivel">
-    <visual>
-      <geometry>
-        <cylinder length="0.065" radius="0.01"/>
-      </geometry>
-      <material name="white">
-        <color rgba="0 0 0 1"/>
-      </material>
-    </visual>
-    <collision>
-      <geometry>
-        <cylinder length="0.065" radius="0.01"/>
-      </geometry>
-    </collision>
-    <inertial>
-      <mass value=".1"/>
-      <xacro:cylinder_intertia length="0.065" radius="0.01" weight="0.1" />
-    </inertial>
-  </link>
-   <joint name="rear_right_swivel_joint" type="continuous">
-    <axis xyz="0 0 1"/>
-    <parent link="right_bar"/>
-    <child link="rear_right_swivel"/>
-    <origin rpy="0 0 0" xyz="${chair_length/2} 0.0 -${chair_height/8}"/>
-    <dynamics damping="0.0" friction="0.5" />
-  </joint>
-  <joint name="rear_right_wheel_joint" type="continuous">
-    <axis xyz="0 0 1"/>
-    <parent link="rear_right_swivel"/>
-    <child link="rear_right_wheel"/>
-    <origin rpy="1.57075 0 0" xyz="0.065 0 0"/>
-    <dynamics damping="0" friction="0.5" />
-  </joint>
-  <link name="rear_right_wheel">
-    <visual>
-      <geometry>
-        <cylinder length="0.05" radius="${small_wheel_radius}"/>
-      </geometry>
-      <material name="white">
-        <color rgba="0 0 0 1"/>
-      </material>
-    </visual>
-    <collision>
-      <geometry>
-        <cylinder length="0.05" radius="${small_wheel_radius}"/>
-      </geometry>
-      <surface>
-        <friction>
-          <ode>
-            <mu>1.0</mu>
-            <mu2>1.0</mu2>
-          </ode>
-        </friction>
-      </surface>
-    </collision>
-    <inertial>
-      <mass value="${small_wheel_weight}"/>
-      <xacro:cylinder_intertia length="${small_wheel_length}" radius="${small_wheel_radius}" weight="${small_wheel_weight}" />
-    </inertial>
-  </link>
-  <link name="rear_left_swivel">
-    <visual>
-      <geometry>
-        <cylinder length="0.065" radius="0.01"/>
-      </geometry>
-      <material name="white">
-        <color rgba="0 0 0 1"/>
-      </material>
-    </visual>
-    <collision>
-      <geometry>
-        <cylinder length="0.065" radius="0.01"/>
-      </geometry>
-    </collision>
-    <inertial>
-      <mass value=".1"/>
-      <xacro:cylinder_intertia length="0.065" radius="0.01" weight="0.1" />
-    </inertial>
-  </link>
-   <joint name="rear_left_swivel_joint" type="continuous">
-    <axis xyz="0 0 1"/>
-    <parent link="left_bar"/>
-    <child link="rear_left_swivel"/>
-    <origin rpy="0 0 0" xyz="${chair_length/2} 0.0 -${chair_height/8}"/>
-    <dynamics damping="0.0" friction="0.5" />
-  </joint>
-  <joint name="rear_left_wheel_joint" type="continuous">
-    <axis xyz="0 0 1"/>
-    <parent link="rear_left_swivel"/>
-    <child link="rear_left_wheel"/>
-    <origin rpy="1.57075 0 0" xyz="0.065 0 0"/>
-    <dynamics damping="0" friction="0.5" />
-  </joint>
-  <link name="rear_left_wheel">
-    <visual>
-      <geometry>
-        <cylinder length="0.05" radius="${small_wheel_radius}"/>
-      </geometry>
-      <material name="white">
-        <color rgba="0 0 0 1"/>
-      </material>
-    </visual>
-    <collision>
-      <geometry>
-        <cylinder length="0.05" radius="${small_wheel_radius}"/>
-      </geometry>
-      <surface>
-        <friction>
-          <ode>
-            <mu>1.0</mu>
-            <mu2>1.0</mu2>
-          </ode>
-        </friction>
-      </surface>
-    </collision>
-    <inertial>
-      <mass value="${small_wheel_weight}"/>
-      <xacro:cylinder_intertia length="${small_wheel_length}" radius="${small_wheel_radius}" weight="${small_wheel_weight}" />
-    </inertial>
-  </link>
 </robot>

Commit message: front point flow odom

File: wheelchair_description/urdf/wheelchair_description_c300.xacro (robot description, xacro)
@@ -2,7 +2,7 @@
 <robot xmlns:xacro="http://www.ros.org/wiki/xacro" name="wheelchair">
   <xacro:property name="PI" value="3.14159265359" />
-  <xacro:property name="chair_width" value="0.643" /> <!-- From front wheel right joint to front wheel left joint -->
-  <xacro:property name="chair_length" value="0.812" /> <!-- From front wheel joint to back wheel joint -->
-  <xacro:property name="chair_height" value="1.191" /> <!-- From front wheel joint to head rest -->
+  <xacro:property name="chair_width" value="0.643" /> <!-- From back wheel right joint to back wheel left joint -->
+  <xacro:property name="chair_length" value="0.812" /> <!-- From back wheel joint to back wheel joint -->
+  <xacro:property name="chair_height" value="1.191" /> <!-- From back wheel joint to head rest -->
   <xacro:property name="chair_weight" value="10.0" />
   <xacro:property name="legs_width" value="0.4064" />
@@ -54,5 +54,5 @@
     </inertial>
   </link>
-  <link name="imu_link">
+  <link name="imu">
     <inertial>
       <mass value="0.01"/>
@@ -69,7 +69,25 @@
   <joint name="imu_joint" type="fixed">
     <parent link="base_link"/>
-    <child link="imu_link"/>
-    <origin xyz="0 0 0" rpy="${PI} 0 0"/>
-  </joint>
+    <child link="imu"/>
+    <origin xyz="0 0 0" rpy="0 0 ${PI}"/>
+  </joint>
+  <link name="flow_sensor">
+      <inertial>
+        <mass value="0.01"/>
+        <origin xyz="0 0 0"/>
+        <inertia ixx="1.0E-6" ixy="0" ixz="0" iyy="1.0E-6" iyz="0" izz="1.0E-6"/>
+      </inertial>
+      <visual>
+        <origin rpy="0 0 0" xyz="0 0 0"/>
+        <geometry>
+          <box size="0.01 0.01 0.01"/>
+        </geometry>
+      </visual>
+    </link>
+    <joint name="flow_joint" type="fixed">
+      <parent link="base_link"/>
+      <child link="flow_sensor"/>
+      <origin xyz="0.5 0 0" rpy="0 0 0"/>
+    </joint>
 <!--Legs -->
   <link name="legs">
@@ -99,4 +117,30 @@
   </joint>
 <!--Right Bar -->
+  <link name="left_bar">
+    <visual>
+      <geometry>
+        <box size="${chair_length + chair_length/4} ${chair_width/4} ${chair_height/8}"/>
+      </geometry>
+      <material name="white">
+        <color rgba="1 1 1 1"/>
+      </material>
+    </visual>
+    <collision>
+      <geometry>
+        <box size="${chair_length + chair_length/4} ${chair_width/4} ${chair_height/8}"/>
+      </geometry>
+    </collision>
+    <inertial>
+      <mass value="2.0"/>
+      <inertia ixx="1e-3" ixy="1e-3" ixz="1e-3" iyy="1e-3" iyz="1e-3" izz="1e-3"/>
+    </inertial>
+  </link>
+  <joint name="left_bar_joint" type="fixed">
+    <axis xyz="0 0 0"/>
+    <parent link="base_link"/>
+    <child link="left_bar"/>
+    <origin rpy="0 0 0" xyz="0.0 ${chair_width/2} -${chair_height/4 + chair_height/8}"/> <!--chair_height/4 + chair_height/8 because this is relative to the center of the bar -->
+  </joint>
+<!--Left Bar -->
   <link name="right_bar">
     <visual>
@@ -122,33 +166,32 @@
     <parent link="base_link"/>
     <child link="right_bar"/>
-    <origin rpy="0 0 0" xyz="0.0 ${chair_width/2} -${chair_height/4 + chair_height/8}"/> <!--chair_height/4 + chair_height/8 because this is relative to the center of the bar -->
-  </joint>
-<!--Left Bar -->
-  <link name="left_bar">
-    <visual>
-      <geometry>
-        <box size="${chair_length + chair_length/4} ${chair_width/4} ${chair_height/8}"/>
-      </geometry>
-      <material name="white">
-        <color rgba="1 1 1 1"/>
-      </material>
-    </visual>
-    <collision>
-      <geometry>
-        <box size="${chair_length + chair_length/4} ${chair_width/4} ${chair_height/8}"/>
-      </geometry>
-    </collision>
-    <inertial>
-      <mass value="2.0"/>
-      <inertia ixx="1e-3" ixy="1e-3" ixz="1e-3" iyy="1e-3" iyz="1e-3" izz="1e-3"/>
-    </inertial>
-  </link>
-  <joint name="left_bar_joint" type="fixed">
-    <axis xyz="0 0 0"/>
-    <parent link="base_link"/>
-    <child link="left_bar"/>
     <origin rpy="0 0 0" xyz="0.0 -${chair_width/2} -${chair_height/4 + chair_height/8}"/> <!--chair_height/4 + chair_height/8 because this is relative to the center of the bar -->
   </joint>
 <!--Main Wheels -->
+  <joint name="left_main_wheel_joint" type="continuous">
+    <axis xyz="0 0 -1"/>
+    <parent link="left_bar"/>
+    <child link="left_main_wheel"/>
+    <origin rpy="1.57075 0 0" xyz="0.2 0.0 -${chair_height/8-0.076}"/>
+  </joint>
+  <link name="left_main_wheel">
+    <visual>
+      <geometry>
+        <cylinder length="${main_wheel_length}" radius="${main_wheel_radius}"/>
+      </geometry>
+      <material name="white">
+        <color rgba="0 0 0 1"/>
+      </material>
+    </visual>
+    <collision>
+      <geometry>
+        <cylinder length="${main_wheel_length}" radius="${main_wheel_radius}"/>
+      </geometry>
+    </collision>
+    <inertial>
+      <mass value="${main_wheel_weight}"/>
+      <xacro:cylinder_intertia length="${main_wheel_length}" radius="${main_wheel_radius}" weight="${main_wheel_weight}" />
+    </inertial>
+  </link>
   <joint name="right_main_wheel_joint" type="continuous">
     <axis xyz="0 0 -1"/>
@@ -176,31 +219,6 @@
     </inertial>
   </link>
-  <joint name="left_main_wheel_joint" type="continuous">
-    <axis xyz="0 0 -1"/>
-    <parent link="left_bar"/>
-    <child link="left_main_wheel"/>
-    <origin rpy="1.57075 0 0" xyz="0.2 0.0 -${chair_height/8-0.076}"/>
-  </joint>
-  <link name="left_main_wheel">
-    <visual>
-      <geometry>
-        <cylinder length="${main_wheel_length}" radius="${main_wheel_radius}"/>
-      </geometry>
-      <material name="white">
-        <color rgba="0 0 0 1"/>
-      </material>
-    </visual>
-    <collision>
-      <geometry>
-        <cylinder length="${main_wheel_length}" radius="${main_wheel_radius}"/>
-      </geometry>
-    </collision>
-    <inertial>
-      <mass value="${main_wheel_weight}"/>
-      <xacro:cylinder_intertia length="${main_wheel_length}" radius="${main_wheel_radius}" weight="${main_wheel_weight}" />
-    </inertial>
-  </link>
 <!--Laser Scanners -->
-  <link name="right_scanner">
+  <link name="left_scanner">
     <visual>
       <origin xyz="0.0 0 0" rpy="0 0 0"/>
@@ -219,35 +237,35 @@
     </inertial>
   </link>
+  <joint name="left_scanner_joint" type="fixed">
+    <axis xyz="0 0 0" />
+    <origin xyz="${chair_length/2 - 0.05/2 + chair_length/8} -${0.05/2} ${chair_height/16 + 0.05}" rpy="0 0 1.5707"/>
+    <parent link="left_bar"/>
+    <child link="right_scanner"/> <!-- TODO UNDO THIS! -->
+  </joint>
+  <link name="right_scanner">
+    <visual>
+      <origin xyz="0.0 0 0" rpy="0 0 0"/>
+      <geometry>
+        <box size="0.05 0.05 0.1"/>
+      </geometry>
+    </visual>
+    <collision>
+      <geometry>
+        <box size="0.05 0.05 0.1"/>
+      </geometry>
+    </collision>
+    <inertial>
+      <mass value="1e-5" />
+      <inertia ixx="1e-3" ixy="0" ixz="0" iyy="1e-3" iyz="0" izz="1e-3" />
+    </inertial>
+  </link>
   <joint name="right_scanner_joint" type="fixed">
     <axis xyz="0 0 0" />
-    <origin xyz="${chair_length/2 - 0.05/2 + chair_length/8} -${0.05/2} ${chair_height/16 + 0.05}" rpy="0 0 1.5707"/>
+    <origin xyz="${chair_length/2 - 0.05/2 + chair_length/8} -${0.05/2} ${chair_height/16 + 0.05}" rpy="0 0 -1.5707"/>
     <parent link="right_bar"/>
-    <child link="right_scanner"/>
-  </joint>
-  <link name="left_scanner">
-    <visual>
-      <origin xyz="0.0 0 0" rpy="0 0 0"/>
-      <geometry>
-        <box size="0.05 0.05 0.1"/>
-      </geometry>
-    </visual>
-    <collision>
-      <geometry>
-        <box size="0.05 0.05 0.1"/>
-      </geometry>
-    </collision>
-    <inertial>
-      <mass value="1e-5" />
-      <inertia ixx="1e-3" ixy="0" ixz="0" iyy="1e-3" iyz="0" izz="1e-3" />
-    </inertial>
-  </link>
-  <joint name="left_scanner_joint" type="fixed">
-    <axis xyz="0 0 0" />
-    <origin xyz="${chair_length/2 - 0.05/2 + chair_length/8} -${0.05/2} ${chair_height/16 + 0.05}" rpy="0 0 -1.5707"/>
-    <parent link="left_bar"/>
-    <child link="left_scanner"/>
-  </joint>
-<!--Front Wheels -->
-  <link name="front_right_swivel">
+    <child link="left_scanner"/> <!-- TODO UNDO THIS! -->
+  </joint>
+<!--back Wheels -->
+  <link name="back_left_swivel">
     <visual>
       <geometry>
@@ -268,19 +286,19 @@
     </inertial>
   </link>
-   <joint name="front_right_swivel_joint" type="continuous">
+   <joint name="back_left_swivel_joint" type="continuous">
     <axis xyz="0 0 1"/>
-    <parent link="right_bar"/>
-    <child link="front_right_swivel"/>
+    <parent link="left_bar"/>
+    <child link="back_left_swivel"/>
     <origin rpy="0 0 0" xyz="-${chair_length/2} 0.0 -${chair_height/8}"/>
     <dynamics damping="0.0" friction="0.5" />
   </joint>
-  <joint name="front_right_wheel_joint" type="continuous">
+  <joint name="back_left_wheel_joint" type="continuous">
     <axis xyz="0 0 1"/>
-    <parent link="front_right_swivel"/>
-    <child link="front_right_wheel"/>
+    <parent link="back_left_swivel"/>
+    <child link="back_left_wheel"/>
     <origin rpy="1.57075 0 0" xyz="0.065 0 0"/>
     <dynamics damping="0" friction="0.5" />
   </joint>
-  <link name="front_right_wheel">
+  <link name="back_left_wheel">
     <visual>
       <geometry>
@@ -309,5 +327,5 @@
     </inertial>
   </link>
-  <link name="front_left_swivel">
+  <link name="back_right_swivel">
     <visual>
       <geometry>
@@ -328,19 +346,19 @@
     </inertial>
   </link>
-   <joint name="front_left_swivel_joint" type="continuous">
+   <joint name="back_right_swivel_joint" type="continuous">
     <axis xyz="0 0 1"/>
-    <parent link="left_bar"/>
-    <child link="front_left_swivel"/>
+    <parent link="right_bar"/>
+    <child link="back_right_swivel"/>
     <origin rpy="0 0 0" xyz="-${chair_length/2} 0.0 -${chair_height/8}"/>
     <dynamics damping="0.0" friction="0.5" />
   </joint>
-  <joint name="front_left_wheel_joint" type="continuous">
+  <joint name="back_right_wheel_joint" type="continuous">
     <axis xyz="0 0 1"/>
-    <parent link="front_left_swivel"/>
-    <child link="front_left_wheel"/>
+    <parent link="back_right_swivel"/>
+    <child link="back_right_wheel"/>
     <origin rpy="1.57075 0 0" xyz="0.065 0 0"/>
     <dynamics damping="0" friction="0.5" />
   </joint>
-  <link name="front_left_wheel">
+  <link name="back_right_wheel">
     <visual>
       <geometry>

File: wheelchair_description/urdf/wheelchair_gazebo.xacro (robot description, xacro)
@@ -15,5 +15,5 @@
     <odometryFrame>odom_temp</odometryFrame>
     <robotBaseFrame>base_footprint</robotBaseFrame>
-    <publishTf>0</publishTf>
+    <publishTf>1</publishTf>
   </plugin>
 </gazebo>

File: wheelchair_description/urdf/wheelchair_gazebo_c300.xacro (robot description, xacro)
@@ -2,10 +2,17 @@
 <robot xmlns:xacro="http://www.ros.org/wiki/xacro" name="wheelchair">
 <xacro:include filename="$(find wheelchair_description)/urdf/wheelchair_description_c300.xacro" />
+<xacro:property name="laser_min" value="0.20" />
+<xacro:property name="laser_max" value="5.599999904632568" />
+<xacro:property name="laser_min_angle" value="-1.5707963705062866" />
+<xacro:property name="laser_max_angle" value="1.5646604299545288" />
+<xacro:property name="laser_update_rate" value="10" />
+<xacro:property name="laser_n_samples" value="512" />
 <gazebo>
   <plugin name="differential_drive_controller" filename="libgazebo_ros_diff_drive.so">
     <alwaysOn>true</alwaysOn>
     <updateRate>50</updateRate>
-    <leftJoint>left_main_wheel_joint</leftJoint>
-    <rightJoint>right_main_wheel_joint</rightJoint>
+    <!-- don't know why these need to be reversed -->
+    <leftJoint>right_main_wheel_joint</leftJoint>
+    <rightJoint>left_main_wheel_joint</rightJoint>
     <wheelSeparation>${chair_width}</wheelSeparation>
     <wheelDiameter>${main_wheel_radius*2}</wheelDiameter>
@@ -15,13 +22,13 @@
     <odometryFrame>odom_temp</odometryFrame>
     <robotBaseFrame>base_footprint</robotBaseFrame>
-    <publishTf>0</publishTf>
+    <publishTf>1</publishTf>
   </plugin>
 </gazebo>
 <gazebo>
   <plugin name="quadrotor_imu_sim" filename="libhector_gazebo_ros_imu.so">
-    <updateRate>50.0</updateRate>
-    <bodyName>imu_link</bodyName>
-    <frameId>imu_link</frameId>
-    <topicName>imu/data</topicName>
+    <updateRate>250.0</updateRate>
+    <bodyName>imu</bodyName>
+    <frameId>imu</frameId>
+    <topicName>/imu/data</topicName>
     <rpyOffsets>0 0 0</rpyOffsets> <!-- deprecated -->
     <gaussianNoise>0</gaussianNoise>  <!-- deprecated -->
@@ -38,17 +45,17 @@
       <pose>0 0 0 0 0 0</pose>
       <visualize>false</visualize>
-      <update_rate>40</update_rate>
+      <update_rate>${laser_update_rate}</update_rate>
       <ray>
         <scan>
           <horizontal>
-            <samples>720</samples>
+            <samples>${laser_n_samples}</samples>
             <resolution>1</resolution>
-            <min_angle>0</min_angle>
-            <max_angle>3.14159265359</max_angle>
+            <min_angle>${laser_min_angle}</min_angle>
+            <max_angle>${laser_max_angle}</max_angle>
           </horizontal>
         </scan>
         <range>
-          <min>2</min>
-          <max>30.0</max>
+          <min>${laser_min}</min>
+          <max>${laser_max}</max>
           <resolution>0.01</resolution>
         </range>
@@ -69,17 +76,17 @@
       <pose>0 0 0 0 0 0</pose>
       <visualize>false</visualize>
-      <update_rate>40</update_rate>
+      <update_rate>${laser_update_rate}</update_rate>
       <ray>
         <scan>
           <horizontal>
-            <samples>720</samples>
+            <samples>${laser_n_samples}</samples>
             <resolution>1</resolution>
-            <min_angle>0</min_angle>
-            <max_angle>3.14159265359</max_angle>
+            <min_angle>${laser_min_angle}</min_angle>
+            <max_angle>${laser_max_angle}</max_angle>
           </horizontal>
         </scan>
         <range>
-          <min>2</min>
-          <max>30.0</max>
+          <min>${laser_min}</min>
+          <max>${laser_max}</max>
           <resolution>0.01</resolution>
         </range>
