Commit message: Updated wheelchair URDF and added IMU sensor

File: wheelchair_description/urdf/modelOld.urdf (robot description, URDF)
Before this commit: robot wheelchair, 18 links, 17 joints
Links:
- link base_footprint: geometry visual box size=0.001 0.001 0.001
- link base_link: geometry collision box size=0.812 0.643 1.191; visual box size=0.812 0.643 1.191
- link front_left_swivel: geometry collision cylinder length=0.065 radius=0.01; visual cylinder length=0.065 radius=0.01
- link front_left_wheel: geometry collision cylinder length=0.05 radius=0.089; visual cylinder length=0.05 radius=0.089
- link front_right_swivel: geometry collision cylinder length=0.065 radius=0.01; visual cylinder length=0.065 radius=0.01
- link front_right_wheel: geometry collision cylinder length=0.05 radius=0.089; visual cylinder length=0.05 radius=0.089
- link imu_link: geometry visual box size=0.01 0.01 0.01
- link left_bar: geometry collision box size=1.015 0.16075 0.148875; visual box size=1.015 0.16075 0.148875
- link left_main_wheel: geometry collision cylinder length=0.065 radius=0.165; visual cylinder length=0.065 radius=0.165
- link left_scanner: geometry collision box size=0.05 0.05 0.1; visual box size=0.05 0.05 0.1
- link legs: geometry collision box size=0.4064 0.4064 0.4064; visual box size=0.4064 0.4064 0.4064
- link rear_left_swivel: geometry collision cylinder length=0.065 radius=0.01; visual cylinder length=0.065 radius=0.01
- link rear_left_wheel: geometry collision cylinder length=0.05 radius=0.089; visual cylinder length=0.05 radius=0.089
- link rear_right_swivel: geometry collision cylinder length=0.065 radius=0.01; visual cylinder length=0.065 radius=0.01
- link rear_right_wheel: geometry collision cylinder length=0.05 radius=0.089; visual cylinder length=0.05 radius=0.089
- link right_bar: geometry collision box size=1.015 0.16075 0.148875; visual box size=1.015 0.16075 0.148875
- link right_main_wheel: geometry collision cylinder length=0.065 radius=0.165; visual cylinder length=0.065 radius=0.165
- link right_scanner: geometry collision box size=0.05 0.05 0.1; visual box size=0.05 0.05 0.1
Joints:
- joint base_footprint_joint: origin xyz= 0 0 .7 rpy=0 0 0 -> xyz= 0 0 0.7 rpy=0 0 0
- joint imu_joint: origin xyz=.32 0 -.35 rpy=3.14159265359 0 0 -> xyz=0 0 0 rpy=3.14159265359 0 0

File: wheelchair_description/urdf/wheelchair_descriptionOld.xacro (robot description, xacro)
@@ -23,8 +23,14 @@
   </xacro:macro>
   <link name="base_footprint">
-    <origin xyz="0 0 .1" rpy="0 0 0"/>
+    <visual>
+      <origin xyz="0 0 0" rpy="0 0 0" />
+        <geometry>
+    	  <!-- <mesh filename="package://wheelchair_description/meshes/wheelchair_rot.dae" scale="0.20 0.20 0.20"/> -->
+          <box size="0.001 0.001 0.001" />
+      </geometry>
+    </visual>
   </link>
   <joint name="base_footprint_joint" type="fixed">
-    <origin xyz=" 0 0 .7" rpy="0 0 0"/>
+    <origin xyz=" 0 0 0.7" rpy="0 0 0"/>
     <parent link="base_footprint"/>
     <child link="base_link"/>
@@ -32,20 +38,17 @@
   <link name="base_link">
     <visual>
-      <origin xyz="0 0 -.59" rpy="0 0 -1.571" />
-        <geometry>
-    	    <mesh filename="package://wheelchair_description/meshes/Wheel_Chair.dae" scale="0.20 0.20 0.20"/>
-      </geometry>
-      <material name="white">
-        <color rgba="1 1 0 .01"/>
-      </material>
-    </visual>
-    <collision>
-      <origin xyz="0 0 -.59" rpy="0 0 -1.571" />
-      <geometry>
-        <mesh filename="package://wheelchair_description/meshes/Wheel_Chair.dae" scale="0.20 0.20 0.20"/>
-      </geometry>
-    </collision>
-    <inertial>
-      <origin xyz="0 0 -.59" rpy="0 0 -1.571" />
+      <geometry>
+        <box size="${chair_length} ${chair_width} ${chair_height}"/>
+      </geometry>
+      <material name="white">
+        <color rgba="1 1 1 1"/>
+      </material>
+    </visual>
+    <collision>
+      <geometry>
+        <box size="${chair_length} ${chair_width} ${chair_height}"/>
+      </geometry>
+    </collision>
+    <inertial>
       <mass value="${chair_weight}"/>
       <xacro:box_intertia height="${chair_height}" length="${chair_length}" width="${chair_width}" weight="${chair_weight}" />
@@ -61,5 +64,5 @@
       <origin rpy="0 0 0" xyz="0 0 0"/>
       <geometry>
-        <box size="0.15 0.1 0.06"/>
+        <box size="0.01 0.01 0.01"/>
       </geometry>
     </visual>
@@ -68,8 +71,21 @@
     <parent link="base_link"/>
     <child link="imu_link"/>
-    <origin xyz=".32 0 -.35" rpy="${PI} 0 0"/>
+    <origin xyz="0 0 0" rpy="${PI} 0 0"/>
   </joint>
 <!--Legs -->
   <link name="legs">
+    <visual>
+      <geometry>
+        <box size="${legs_length} ${legs_width} ${legs_height}"/>
+      </geometry>
+      <material name="white">
+        <color rgba="1 1 1 1"/>
+      </material>
+    </visual>
+    <collision>
+      <geometry>
+        <box size="${legs_length} ${legs_width} ${legs_height}"/>
+      </geometry>
+    </collision>
     <inertial>
       <mass value="${legs_weight}"/>
@@ -77,5 +93,5 @@
     </inertial>
   </link>
-  <joint name="legs_joint" type="fixed">
+    <joint name="legs_joint" type="fixed">
     <axis xyz="0 0 0"/>
     <parent link="base_link"/>
@@ -85,4 +101,17 @@
 <!--Right Bar -->
   <link name="right_bar">
+    <visual>
+      <geometry>
+        <box size="${chair_length + chair_length/4} ${chair_width/4} ${chair_height/8}"/>
+      </geometry>
+      <material name="white">
+        <color rgba="1 1 1 1"/>
+      </material>
+    </visual>
+    <collision>
+      <geometry>
+        <box size="${chair_length + chair_length/4} ${chair_width/4} ${chair_height/8}"/>
+      </geometry>
+    </collision>
     <inertial>
       <mass value="2.0"/>
@@ -98,4 +127,17 @@
 <!--Left Bar -->
   <link name="left_bar">
+    <visual>
+      <geometry>
+        <box size="${chair_length + chair_length/4} ${chair_width/4} ${chair_height/8}"/>
+      </geometry>
+      <material name="white">
+        <color rgba="1 1 1 1"/>
+      </material>
+    </visual>
+    <collision>
+      <geometry>
+        <box size="${chair_length + chair_length/4} ${chair_width/4} ${chair_height/8}"/>
+      </geometry>
+    </collision>
     <inertial>
       <mass value="2.0"/>
@@ -117,4 +159,12 @@
   </joint>
   <link name="right_main_wheel">
+    <visual>
+      <geometry>
+        <cylinder length="${main_wheel_length}" radius="${main_wheel_radius}"/>
+      </geometry>
+      <material name="white">
+        <color rgba="0 0 0 1"/>
+      </material>
+    </visual>
     <collision>
       <geometry>
@@ -134,4 +184,12 @@
   </joint>
   <link name="left_main_wheel">
+    <visual>
+      <geometry>
+        <cylinder length="${main_wheel_length}" radius="${main_wheel_radius}"/>
+      </geometry>
+      <material name="white">
+        <color rgba="0 0 0 1"/>
+      </material>
+    </visual>
     <collision>
       <geometry>
@@ -146,4 +204,15 @@
 <!--Laser Scanners -->
   <link name="right_scanner">
+    <visual>
+      <origin xyz="0.0 0 0" rpy="0 0 0"/>
+      <geometry>
+        <box size="0.05 0.05 0.1"/>
+      </geometry>
+    </visual>
+    <collision>
+      <geometry>
+        <box size="0.05 0.05 0.1"/>
+      </geometry>
+    </collision>
     <inertial>
       <mass value="1e-5" />
@@ -158,4 +227,15 @@
   </joint>
   <link name="left_scanner">
+    <visual>
+      <origin xyz="0.0 0 0" rpy="0 0 0"/>
+      <geometry>
+        <box size="0.05 0.05 0.1"/>
+      </geometry>
+    </visual>
+    <collision>
+      <geometry>
+        <box size="0.05 0.05 0.1"/>
+      </geometry>
+    </collision>
     <inertial>
       <mass value="1e-5" />
@@ -171,4 +251,12 @@
 <!--Front Wheels -->
   <link name="front_right_swivel">
+    <visual>
+      <geometry>
+        <cylinder length="0.065" radius="0.01"/>
+      </geometry>
+      <material name="white">
+        <color rgba="0 0 0 1"/>
+      </material>
+    </visual>
     <collision>
       <geometry>
@@ -196,4 +284,12 @@
   </joint>
   <link name="front_right_wheel">
+    <visual>
+      <geometry>
+        <cylinder length="${small_wheel_length}" radius="${small_wheel_radius}"/>
+      </geometry>
+      <material name="white">
+        <color rgba="0 0 0 1"/>
+      </material>
+    </visual>
     <collision>
       <geometry>
@@ -215,4 +311,12 @@
   </link>
   <link name="front_left_swivel">
+    <visual>
+      <geometry>
+        <cylinder length="0.065" radius="0.01"/>
+      </geometry>
+      <material name="white">
+        <color rgba="0 0 0 1"/>
+      </material>
+    </visual>
     <collision>
       <geometry>
@@ -240,4 +344,12 @@
   </joint>
   <link name="front_left_wheel">
+    <visual>
+      <geometry>
+        <cylinder length="0.05" radius="${small_wheel_radius}"/>
+      </geometry>
+      <material name="white">
+        <color rgba="0 0 0 1"/>
+      </material>
+    </visual>
     <collision>
       <geometry>
@@ -260,4 +372,12 @@
 <!--Rear Wheels -->
   <link name="rear_right_swivel">
+    <visual>
+      <geometry>
+        <cylinder length="0.065" radius="0.01"/>
+      </geometry>
+      <material name="white">
+        <color rgba="0 0 0 1"/>
+      </material>
+    </visual>
     <collision>
       <geometry>
@@ -285,4 +405,12 @@
   </joint>
   <link name="rear_right_wheel">
+    <visual>
+      <geometry>
+        <cylinder length="0.05" radius="${small_wheel_radius}"/>
+      </geometry>
+      <material name="white">
+        <color rgba="0 0 0 1"/>
+      </material>
+    </visual>
     <collision>
       <geometry>
@@ -304,4 +432,12 @@
   </link>
   <link name="rear_left_swivel">
+    <visual>
+      <geometry>
+        <cylinder length="0.065" radius="0.01"/>
+      </geometry>
+      <material name="white">
+        <color rgba="0 0 0 1"/>
+      </material>
+    </visual>
     <collision>
       <geometry>
@@ -329,4 +465,12 @@
   </joint>
   <link name="rear_left_wheel">
+    <visual>
+      <geometry>
+        <cylinder length="0.05" radius="${small_wheel_radius}"/>
+      </geometry>
+      <material name="white">
+        <color rgba="0 0 0 1"/>
+      </material>
+    </visual>
     <collision>
       <geometry>
@@ -347,25 +491,3 @@
     </inertial>
   </link>
-  <gazebo>
-    <plugin name="gazebo_ros_control" filename="libgazebo_ros_control.so">
-      <robotNamespace>/</robotNamespace>
-    </plugin>
-  </gazebo>
-  <gazebo reference="imu_link">
-    <sensor name="imu_sensor" type="imu">
-      <always_on>true</always_on>
-      <update_rate>100</update_rate>
-      <visualize>true</visualize>
-      <topic>__default_topic__</topic>
-      <plugin name="imu_plugin" filename="libgazebo_ros_imu_sensor.so">
-        <topicName>imu</topicName>
-        <bodyName>imu_link</bodyName>
-        <updateRateHZ>10.0</updateRateHZ>
-        <gaussianNoise>0.0</gaussianNoise>
-        <xyzOffset>0 0 0</xyzOffset>
-        <rpyOffset>0 0 0</rpyOffset>
-        <frameName>imu_link</frameName>
-      </plugin>
-    </sensor>
-  </gazebo>
 </robot>

File: wheelchair_description/urdf/wheelchair_description_mesh_physics.xacro (robot description, xacro)
@@ -32,5 +32,5 @@
   <link name="base_link">
     <visual>
-      <origin xyz="0 0 -.59" rpy="0 0 -1.571" />
+      <origin xyz="0 0 -.605" rpy="0 0 -1.571" />
         <geometry>
     	    <mesh filename="package://wheelchair_description/meshes/Wheel_Chair.dae" scale="0.20 0.20 0.20"/>
@@ -41,5 +41,5 @@
     </visual>
     <collision>
-      <origin xyz="0 0 -.59" rpy="0 0 -1.571" />
+      <origin xyz="0 0 -.605" rpy="0 0 -1.571" />
       <geometry>
         <mesh filename="package://wheelchair_description/meshes/Wheel_Chair.dae" scale="0.20 0.20 0.20"/>
@@ -47,5 +47,5 @@
     </collision>
     <inertial>
-      <origin xyz="0 0 -.59" rpy="0 0 -1.571" />
+      <origin xyz="0 0 -.605" rpy="0 0 -1.571" />
       <mass value="${chair_weight}"/>
       <xacro:box_intertia height="${chair_height}" length="${chair_length}" width="${chair_width}" weight="${chair_weight}" />
@@ -61,5 +61,5 @@
       <origin rpy="0 0 0" xyz="0 0 0"/>
       <geometry>
-        <box size="0.15 0.1 0.06"/>
+        <box size="0.001 0.001 0.001"/>
       </geometry>
     </visual>
@@ -68,5 +68,5 @@
     <parent link="base_link"/>
     <child link="imu_link"/>
-    <origin xyz=".32 0 -.35" rpy="${PI} 0 0"/>
+    <origin xyz="0 0 0" rpy="${PI} 0 0"/>
   </joint>
 <!--Legs -->
@@ -347,25 +347,3 @@
     </inertial>
   </link>
-  <gazebo>
-    <plugin name="gazebo_ros_control" filename="libgazebo_ros_control.so">
-      <robotNamespace>/</robotNamespace>
-    </plugin>
-  </gazebo>
-  <gazebo reference="imu_link">
-    <sensor name="imu_sensor" type="imu">
-      <always_on>true</always_on>
-      <update_rate>100</update_rate>
-      <visualize>true</visualize>
-      <topic>__default_topic__</topic>
-      <plugin name="imu_plugin" filename="libgazebo_ros_imu_sensor.so">
-        <topicName>imu</topicName>
-        <bodyName>imu_link</bodyName>
-        <updateRateHZ>10.0</updateRateHZ>
-        <gaussianNoise>0.0</gaussianNoise>
-        <xyzOffset>0 0 0</xyzOffset>
-        <rpyOffset>0 0 0</rpyOffset>
-        <frameName>imu_link</frameName>
-      </plugin>
-    </sensor>
-  </gazebo>
 </robot>

File: wheelchair_description/urdf/wheelchair_description_mesh_visuals.xacro (robot description, xacro)
@@ -23,8 +23,14 @@
   </xacro:macro>
   <link name="base_footprint">
-    <origin xyz="0 0 .1" rpy="0 0 0"/>
+    <visual>
+      <origin xyz="0 0 .1" rpy="0 0 -1.571" />
+        <geometry>
+    	    <mesh filename="package://wheelchair_description/meshes/Wheel_Chair.dae" scale="0.20 0.20 0.20"/>
+          <!--<box size="0.001 0.001 0.001" />-->
+      </geometry>
+    </visual>
   </link>
   <joint name="base_footprint_joint" type="fixed">
-    <origin xyz=" 0 0 .7" rpy="0 0 0"/>
+    <origin xyz=" 0 0 0.7" rpy="0 0 0"/>
     <parent link="base_footprint"/>
     <child link="base_link"/>
@@ -32,7 +38,7 @@
   <link name="base_link">
     <visual>
-      <origin xyz="0 0 -.59" rpy="0 0 -1.571" />
-        <geometry>
-    	    <mesh filename="package://wheelchair_description/meshes/Wheel_Chair.dae" scale="0.20 0.20 0.20"/>
+      <geometry>
+        <!--<mesh filename="package://wheelchair_description/meshes/Wheel_Chair.dae" scale="0.20 0.20 0.20"/>-->
+        <box size=".001 .001 .001"/>
       </geometry>
       <material name="white">
@@ -41,11 +47,9 @@
     </visual>
     <collision>
-      <origin xyz="0 0 -.59" rpy="0 0 -1.571" />
-      <geometry>
-        <mesh filename="package://wheelchair_description/meshes/Wheel_Chair.dae" scale="0.20 0.20 0.20"/>
-      </geometry>
-    </collision>
-    <inertial>
-      <origin xyz="0 0 -.59" rpy="0 0 -1.571" />
+      <geometry>
+        <box size="${chair_length} ${chair_width} ${chair_height}"/>
+      </geometry>
+    </collision>
+    <inertial>
       <mass value="${chair_weight}"/>
       <xacro:box_intertia height="${chair_height}" length="${chair_length}" width="${chair_width}" weight="${chair_weight}" />
@@ -61,5 +65,5 @@
       <origin rpy="0 0 0" xyz="0 0 0"/>
       <geometry>
-        <box size="0.15 0.1 0.06"/>
+        <box size="0.001 0.001 0.001"/>
       </geometry>
     </visual>
@@ -68,8 +72,21 @@
     <parent link="base_link"/>
     <child link="imu_link"/>
-    <origin xyz=".32 0 -.35" rpy="${PI} 0 0"/>
+    <origin xyz="0 0 0" rpy="${PI} 0 0"/>
   </joint>
 <!--Legs -->
   <link name="legs">
+    <visual>
+      <geometry>
+        <box size=".001 .001 .001"/>
+      </geometry>
+      <material name="white">
+        <color rgba="1 1 1 .01"/>
+      </material>
+    </visual>
+    <collision>
+      <geometry>
+        <box size="${legs_length} ${legs_width} ${legs_height}"/>
+      </geometry>
+    </collision>
     <inertial>
       <mass value="${legs_weight}"/>
@@ -77,5 +94,5 @@
     </inertial>
   </link>
-  <joint name="legs_joint" type="fixed">
+    <joint name="legs_joint" type="fixed">
     <axis xyz="0 0 0"/>
     <parent link="base_link"/>
@@ -85,4 +102,17 @@
 <!--Right Bar -->
   <link name="right_bar">
+    <visual>
+      <geometry>
+        <box size=".001 .001 .001"/>
+      </geometry>
+      <material name="white">
+        <color rgba="1 1 1 .01"/>
+      </material>
+    </visual>
+    <collision>
+      <geometry>
+        <box size="${chair_length + chair_length/4} ${chair_width/4} ${chair_height/8}"/>
+      </geometry>
+    </collision>
     <inertial>
       <mass value="2.0"/>
@@ -98,4 +128,17 @@
 <!--Left Bar -->
   <link name="left_bar">
+    <visual>
+      <geometry>
+        <box size=".001 .001 .001"/>
+      </geometry>
+      <material name="white">
+        <color rgba="1 1 1 .01"/>
+      </material>
+    </visual>
+    <collision>
+      <geometry>
+        <box size="${chair_length + chair_length/4} ${chair_width/4} ${chair_height/8}"/>
+      </geometry>
+    </collision>
     <inertial>
       <mass value="2.0"/>
@@ -117,4 +160,12 @@
   </joint>
   <link name="right_main_wheel">
+    <visual>
+      <geometry>
+        <cylinder length=".001" radius=".001"/>
+      </geometry>
+      <material name="white">
+        <color rgba="0 0 0 .01"/>
+      </material>
+    </visual>
     <collision>
       <geometry>
@@ -134,4 +185,12 @@
   </joint>
   <link name="left_main_wheel">
+    <visual>
+      <geometry>
+        <cylinder length=".001" radius=".001"/>
+      </geometry>
+      <material name="white">
+        <color rgba="0 0 0 .01"/>
+      </material>
+    </visual>
     <collision>
       <geometry>
@@ -146,4 +205,15 @@
 <!--Laser Scanners -->
   <link name="right_scanner">
+    <visual>
+      <origin xyz="0.0 0 0" rpy="0 0 0"/>
+      <geometry>
+        <box size="0.001 0.001 0.001"/>
+      </geometry>
+    </visual>
+    <collision>
+      <geometry>
+        <box size="0.05 0.05 0.1"/>
+      </geometry>
+    </collision>
     <inertial>
       <mass value="1e-5" />
@@ -158,4 +228,15 @@
   </joint>
   <link name="left_scanner">
+    <visual>
+      <origin xyz="0.0 0 0" rpy="0 0 0"/>
+      <geometry>
+        <box size="0.001 0.001 0.001"/>
+      </geometry>
+    </visual>
+    <collision>
+      <geometry>
+        <box size="0.05 0.05 0.1"/>
+      </geometry>
+    </collision>
     <inertial>
       <mass value="1e-5" />
@@ -171,4 +252,12 @@
 <!--Front Wheels -->
   <link name="front_right_swivel">
+    <visual>
+      <geometry>
+        <cylinder length="0.001" radius="0.001"/>
+      </geometry>
+      <material name="white">
+        <color rgba="0 0 0 .01"/>
+      </material>
+    </visual>
     <collision>
       <geometry>
@@ -196,4 +285,12 @@
   </joint>
   <link name="front_right_wheel">
+    <visual>
+      <geometry>
+        <cylinder length=".001" radius=".001"/>
+      </geometry>
+      <material name="white">
+        <color rgba="0 0 0 .01"/>
+      </material>
+    </visual>
     <collision>
       <geometry>
@@ -215,4 +312,12 @@
   </link>
   <link name="front_left_swivel">
+    <visual>
+      <geometry>
+        <cylinder length=".001" radius=".001"/>
+      </geometry>
+      <material name="white">
+        <color rgba="0 0 0 .01"/>
+      </material>
+    </visual>
     <collision>
       <geometry>
@@ -240,4 +345,12 @@
   </joint>
   <link name="front_left_wheel">
+    <visual>
+      <geometry>
+        <cylinder length=".001" radius=".001"/>
+      </geometry>
+      <material name="white">
+        <color rgba="0 0 0 .01"/>
+      </material>
+    </visual>
     <collision>
       <geometry>
@@ -260,4 +373,12 @@
 <!--Rear Wheels -->
   <link name="rear_right_swivel">
+    <visual>
+      <geometry>
+        <cylinder length=".001" radius=".001"/>
+      </geometry>
+      <material name="white">
+        <color rgba="0 0 0 .01"/>
+      </material>
+    </visual>
     <collision>
       <geometry>
@@ -285,4 +406,12 @@
   </joint>
   <link name="rear_right_wheel">
+    <visual>
+      <geometry>
+        <cylinder length=".001" radius=".001"/>
+      </geometry>
+      <material name="white">
+        <color rgba="0 0 0 .01"/>
+      </material>
+    </visual>
     <collision>
       <geometry>
@@ -304,4 +433,12 @@
   </link>
   <link name="rear_left_swivel">
+    <visual>
+      <geometry>
+        <cylinder length=".001" radius=".001"/>
+      </geometry>
+      <material name="white">
+        <color rgba="0 0 0 .01"/>
+      </material>
+    </visual>
     <collision>
       <geometry>
@@ -329,4 +466,12 @@
   </joint>
   <link name="rear_left_wheel">
+    <visual>
+      <geometry>
+        <cylinder length=".001" radius=".001"/>
+      </geometry>
+      <material name="white">
+        <color rgba="0 0 0 .01"/>
+      </material>
+    </visual>
     <collision>
       <geometry>
@@ -347,25 +492,3 @@
     </inertial>
   </link>
-  <gazebo>
-    <plugin name="gazebo_ros_control" filename="libgazebo_ros_control.so">
-      <robotNamespace>/</robotNamespace>
-    </plugin>
-  </gazebo>
-  <gazebo reference="imu_link">
-    <sensor name="imu_sensor" type="imu">
-      <always_on>true</always_on>
-      <update_rate>100</update_rate>
-      <visualize>true</visualize>
-      <topic>__default_topic__</topic>
-      <plugin name="imu_plugin" filename="libgazebo_ros_imu_sensor.so">
-        <topicName>imu</topicName>
-        <bodyName>imu_link</bodyName>
-        <updateRateHZ>10.0</updateRateHZ>
-        <gaussianNoise>0.0</gaussianNoise>
-        <xyzOffset>0 0 0</xyzOffset>
-        <rpyOffset>0 0 0</rpyOffset>
-        <frameName>imu_link</frameName>
-      </plugin>
-    </sensor>
-  </gazebo>
 </robot>

File: wheelchair_description/urdf/wheelchair_gazebo.xacro (robot description, xacro)
@@ -10,5 +10,6 @@
     <wheelSeparation>${chair_width}</wheelSeparation>
     <wheelDiameter>${main_wheel_radius*2}</wheelDiameter>
-    <torque>20</torque>
+    <wheelTorque>20</wheelTorque>
+    <wheelAcceleration>1</wheelAcceleration>
     <commandTopic>cmd_vel</commandTopic>
     <odometryTopic>odom_temp</odometryTopic>
@@ -18,5 +19,4 @@
   </plugin>
 </gazebo>
-<!--
 <gazebo>
   <plugin name="quadrotor_imu_sim" filename="libhector_gazebo_ros_imu.so">
@@ -35,5 +35,4 @@
   </plugin>
 </gazebo>
--->
 <gazebo reference="right_scanner">
     <sensor type="ray" name="head_hokuyo_sensor">
