Commit message: Odom issues.

File: wheelchair_description/urdf/wheelchair_description.xacro (robot description, xacro)
@@ -202,5 +202,5 @@
   <joint name="right_scanner_joint" type="fixed">
     <axis xyz="0 0 0" />
-    <origin xyz="${chair_length/2 - 0.05/2 + chair_length/8} -${0.05/2} ${chair_height/16 + 0.05}" rpy="0 0 1.57079632679"/>
+    <origin xyz="${chair_length/2 - 0.05/2 + chair_length/8} -${0.05/2} ${chair_height/16 + 0.05}" rpy="0 0 0"/>
     <parent link="right_bar"/>
     <child link="right_scanner"/>
@@ -225,5 +225,5 @@
   <joint name="left_scanner_joint" type="fixed">
     <axis xyz="0 0 0" />
-    <origin xyz="${chair_length/2 - 0.05/2 + chair_length/8} -${0.05/2} ${chair_height/16 + 0.05}" rpy="0 0 -1.57079632679"/>
+    <origin xyz="${chair_length/2 - 0.05/2 + chair_length/8} -${0.05/2} ${chair_height/16 + 0.05}" rpy="0 0 -3.14159265359"/>
     <parent link="left_bar"/>
     <child link="left_scanner"/>

File: wheelchair_description/urdf/wheelchair_gazebo.xacro (robot description, xacro)
@@ -28,6 +28,6 @@
             <samples>720</samples>
             <resolution>1</resolution>
-            <min_angle>-1.57079632679</min_angle>
-            <max_angle>1.57079632679</max_angle>
+            <min_angle>0</min_angle>
+            <max_angle>3.14159265359</max_angle>
           </horizontal>
         </scan>
@@ -59,6 +59,6 @@
             <samples>720</samples>
             <resolution>1</resolution>
-            <min_angle>-1.57079632679</min_angle>
-            <max_angle>1.57079632679</max_angle>
+            <min_angle>0</min_angle>
+            <max_angle>3.14159265359</max_angle>
           </horizontal>
         </scan>

Commit message: Rotated left/right LIDAR joints 90 degree

File: wheelchair_description/urdf/wheelchair_description.xacro (robot description, xacro)
@@ -202,5 +202,5 @@
   <joint name="right_scanner_joint" type="fixed">
     <axis xyz="0 0 0" />
-    <origin xyz="${chair_length/2 - 0.05/2 + chair_length/8} -${0.05/2} ${chair_height/16 + 0.05}" rpy="0 0 0"/>
+    <origin xyz="${chair_length/2 - 0.05/2 + chair_length/8} -${0.05/2} ${chair_height/16 + 0.05}" rpy="0 0 1.5707"/>
     <parent link="right_bar"/>
     <child link="right_scanner"/>
@@ -225,5 +225,5 @@
   <joint name="left_scanner_joint" type="fixed">
     <axis xyz="0 0 0" />
-    <origin xyz="${chair_length/2 - 0.05/2 + chair_length/8} -${0.05/2} ${chair_height/16 + 0.05}" rpy="0 0 -3.14159265359"/>
+    <origin xyz="${chair_length/2 - 0.05/2 + chair_length/8} -${0.05/2} ${chair_height/16 + 0.05}" rpy="0 0 -1.5707"/>
     <parent link="left_bar"/>
     <child link="left_scanner"/>

Commit message: add IMU

File: wheelchair_description/urdf/wheelchair_description.xacro (robot description, xacro)
@@ -1,4 +1,5 @@
 <?xml version="1.0"?>
 <robot xmlns:xacro="http://www.ros.org/wiki/xacro" name="wheelchair">
+  <xacro:property name="PI" value="3.14159265359" />
   <xacro:property name="chair_width" value="0.643" /> <!-- From front wheel right joint to front wheel left joint -->
   <xacro:property name="chair_length" value="0.812" /> <!-- From front wheel joint to back wheel joint -->
@@ -53,4 +54,22 @@
     </inertial>
   </link>
+  <link name="imu_link">
+    <inertial>
+      <mass value="0.01"/>
+      <origin xyz="0 0 0"/>
+      <inertia ixx="1.0E-6" ixy="0" ixz="0" iyy="1.0E-6" iyz="0" izz="1.0E-6"/>
+    </inertial>
+    <visual>
+      <origin rpy="0 0 0" xyz="0 0 0"/>
+      <geometry>
+        <box size="0.01 0.01 0.01"/>
+      </geometry>
+    </visual>
+  </link>
+  <joint name="imu_joint" type="fixed">
+    <parent link="base_link"/>
+    <child link="imu_link"/>
+    <origin xyz="0 0 0" rpy="${PI} 0 0"/>
+  </joint>
 <!--Legs -->
   <link name="legs">

File: wheelchair_description/urdf/wheelchair_gazebo.xacro (robot description, xacro)
@@ -16,4 +16,20 @@
     <robotBaseFrame>base_footprint</robotBaseFrame>
     <publishTf>0</publishTf>
+  </plugin>
+</gazebo>
+<gazebo>
+  <plugin name="quadrotor_imu_sim" filename="libhector_gazebo_ros_imu.so">
+    <updateRate>50.0</updateRate>
+    <bodyName>imu_link</bodyName>
+    <frameId>imu_link</frameId>
+    <topicName>imu/data</topicName>
+    <rpyOffsets>0 0 0</rpyOffsets> <!-- deprecated -->
+    <gaussianNoise>0</gaussianNoise>  <!-- deprecated -->
+    <accelDrift>0.5 0.5 0.5</accelDrift>
+    <accelGaussianNoise>0.05 0.05 0.05</accelGaussianNoise>
+    <rateDrift>0.1 0.1 0.1</rateDrift>
+    <rateGaussianNoise>0.05 0.05 0.015</rateGaussianNoise>
+    <headingDrift>0.1</headingDrift>
+    <headingGaussianNoise>0.05</headingGaussianNoise>
   </plugin>
 </gazebo>

Commit message: initial checkin for dubai changes

File: wheelchair_description/urdf/wheelchair_description.xacro (robot description, xacro)
@@ -26,4 +26,5 @@
       <origin xyz="0 0 0" rpy="0 0 0" />
         <geometry>
+    	  <!-- <mesh filename="package://wheelchair_description/meshes/wheelchair_rot.dae" scale="0.20 0.20 0.20"/> -->
           <box size="0.001 0.001 0.001" />
       </geometry>
@@ -221,5 +222,5 @@
   <joint name="right_scanner_joint" type="fixed">
     <axis xyz="0 0 0" />
-    <origin xyz="${chair_length/2 - 0.05/2 + chair_length/8} -${0.05/2} ${chair_height/16 + 0.05}" rpy="0 0 1.5707"/>
+    <origin xyz="${chair_length/2 - 0.05/2 + chair_length/8} ${0.05/2} ${chair_height/16 + 0.05}" rpy="0 0 1.5707"/>
     <parent link="right_bar"/>
     <child link="right_scanner"/>

File: wheelchair_description/urdf/wheelchair_gazebo.xacro (robot description, xacro)
@@ -18,4 +18,5 @@
   </plugin>
 </gazebo>
+<!--
 <gazebo>
   <plugin name="quadrotor_imu_sim" filename="libhector_gazebo_ros_imu.so">
@@ -24,6 +25,6 @@
     <frameId>imu_link</frameId>
     <topicName>imu/data</topicName>
-    <rpyOffsets>0 0 0</rpyOffsets> <!-- deprecated -->
-    <gaussianNoise>0</gaussianNoise>  <!-- deprecated -->
+    <rpyOffsets>0 0 0</rpyOffsets>
+    <gaussianNoise>0</gaussianNoise>
     <accelDrift>0.5 0.5 0.5</accelDrift>
     <accelGaussianNoise>0.05 0.05 0.05</accelGaussianNoise>
@@ -34,8 +35,9 @@
   </plugin>
 </gazebo>
+-->
 <gazebo reference="right_scanner">
     <sensor type="ray" name="head_hokuyo_sensor">
       <pose>0 0 0 0 0 0</pose>
-      <visualize>false</visualize>
+      <visualize>true</visualize>
       <update_rate>40</update_rate>
       <ray>
@@ -44,11 +46,11 @@
             <samples>720</samples>
             <resolution>1</resolution>
-            <min_angle>0</min_angle>
-            <max_angle>3.14159265359</max_angle>
+            <min_angle>-2.3561925</min_angle>
+            <max_angle>1.57079</max_angle>
           </horizontal>
         </scan>
         <range>
-          <min>2</min>
-          <max>30.0</max>
+          <min>0.2</min>
+          <max>10.1</max>
           <resolution>0.01</resolution>
         </range>
@@ -56,5 +58,5 @@
           <type>gaussian</type>
           <mean>0.0</mean>
-          <stddev>0.01</stddev>
+          <stddev>0.02</stddev>
         </noise>
       </ray>
@@ -68,5 +70,5 @@
     <sensor type="ray" name="head_hokuyo_sensor2">
       <pose>0 0 0 0 0 0</pose>
-      <visualize>false</visualize>
+      <visualize>true</visualize>
       <update_rate>40</update_rate>
       <ray>
@@ -75,11 +77,11 @@
             <samples>720</samples>
             <resolution>1</resolution>
-            <min_angle>0</min_angle>
-            <max_angle>3.14159265359</max_angle>
+            <min_angle>-1.57079</min_angle>
+            <max_angle>2.3561925</max_angle>
           </horizontal>
         </scan>
         <range>
-          <min>2</min>
-          <max>30.0</max>
+          <min>0.2</min>
+          <max>10.1</max>
           <resolution>0.01</resolution>
         </range>
@@ -87,5 +89,5 @@
           <type>gaussian</type>
           <mean>0.0</mean>
-          <stddev>0.01</stddev>
+          <stddev>0.02</stddev>
         </noise>
       </ray>

Commit message: Adjusted URDF model

File: wheelchair_description/urdf/wheelchair_description.xacro (robot description, xacro)
@@ -153,5 +153,5 @@
   <joint name="right_scanner_joint" type="fixed">
     <axis xyz="0 0 0" />
-    <origin xyz="${chair_length/2 - 0.1/2 + chair_length/8} ${0.05/2 - .025} ${chair_height/16 + 0.05}" rpy="0 0 1.5707"/>
+    <origin xyz="${chair_length/2 - 0.1/2 + chair_length/8} ${0.05/2 - .005} ${chair_height/16 + 0.05}" rpy="0 0 1.5707"/>
     <parent link="right_bar"/>
     <child link="right_scanner"/>
@@ -165,5 +165,5 @@
   <joint name="left_scanner_joint" type="fixed">
     <axis xyz="0 0 0" />
-    <origin xyz="${chair_length/2 - 0.1/2 + chair_length/8} -${0.05/2 - .025} ${chair_height/16 + 0.05}" rpy="0 0 -1.5707"/>
+    <origin xyz="${chair_length/2 - 0.1/2 + chair_length/8} -${0.05/2 - .005} ${chair_height/16 + 0.05}" rpy="0 0 -1.5707"/>
     <parent link="left_bar"/>
     <child link="left_scanner"/>

Commit message: Adjusted URDF model

File: wheelchair_description/urdf/wheelchair_description.xacro (robot description, xacro)
@@ -153,5 +153,5 @@
   <joint name="right_scanner_joint" type="fixed">
     <axis xyz="0 0 0" />
-    <origin xyz="${chair_length/2 - 0.1/2 + chair_length/8} ${0.05/2 - .005} ${chair_height/16 + 0.05}" rpy="0 0 1.5707"/>
+    <origin xyz="${chair_length/2 - 0.1/2 + chair_length/8} ${0.05/2 - .025} ${chair_height/16 + 0.05}" rpy="0 0 1.5707"/>
     <parent link="right_bar"/>
     <child link="right_scanner"/>
@@ -165,5 +165,5 @@
   <joint name="left_scanner_joint" type="fixed">
     <axis xyz="0 0 0" />
-    <origin xyz="${chair_length/2 - 0.1/2 + chair_length/8} -${0.05/2 - .005} ${chair_height/16 + 0.05}" rpy="0 0 -1.5707"/>
+    <origin xyz="${chair_length/2 - 0.1/2 + chair_length/8} -${0.05/2 - .025} ${chair_height/16 + 0.05}" rpy="0 0 -1.5707"/>
     <parent link="left_bar"/>
     <child link="left_scanner"/>

Commit message: Adjusted URDF model

File: wheelchair_description/urdf/wheelchair_description.xacro (robot description, xacro)
@@ -153,5 +153,5 @@
   <joint name="right_scanner_joint" type="fixed">
     <axis xyz="0 0 0" />
-    <origin xyz="${chair_length/2 - 0.1/2 + chair_length/8} ${0.05/2 - .005} ${chair_height/16 + 0.05}" rpy="0 0 1.5707"/>
+    <origin xyz="${chair_length/2 - 0.1/2 + chair_length/8} ${0.05/2 + .005} ${chair_height/16 + 0.05}" rpy="0 0 1.5707"/>
     <parent link="right_bar"/>
     <child link="right_scanner"/>
@@ -165,5 +165,5 @@
   <joint name="left_scanner_joint" type="fixed">
     <axis xyz="0 0 0" />
-    <origin xyz="${chair_length/2 - 0.1/2 + chair_length/8} -${0.05/2 - .005} ${chair_height/16 + 0.05}" rpy="0 0 -1.5707"/>
+    <origin xyz="${chair_length/2 - 0.1/2 + chair_length/8} -${0.05/2 + .005} ${chair_height/16 + 0.05}" rpy="0 0 -1.5707"/>
     <parent link="left_bar"/>
     <child link="left_scanner"/>

Commit message: Adjusted URDF model

File: wheelchair_description/urdf/wheelchair_description.xacro (robot description, xacro)
@@ -153,5 +153,5 @@
   <joint name="right_scanner_joint" type="fixed">
     <axis xyz="0 0 0" />
-    <origin xyz="${chair_length/2 - 0.1/2 + chair_length/8} ${0.05/2 + .005} ${chair_height/16 + 0.05}" rpy="0 0 1.5707"/>
+    <origin xyz="${chair_length/2 - 0.1/2 + chair_length/8} -${0.05/2 + .12} ${chair_height/16 + 0.05}" rpy="0 0 1.5707"/>
     <parent link="right_bar"/>
     <child link="right_scanner"/>
@@ -165,5 +165,5 @@
   <joint name="left_scanner_joint" type="fixed">
     <axis xyz="0 0 0" />
-    <origin xyz="${chair_length/2 - 0.1/2 + chair_length/8} -${0.05/2 + .005} ${chair_height/16 + 0.05}" rpy="0 0 -1.5707"/>
+    <origin xyz="${chair_length/2 - 0.1/2 + chair_length/8} ${0.05/2 + .12} ${chair_height/16 + 0.05}" rpy="0 0 -1.5707"/>
     <parent link="left_bar"/>
     <child link="left_scanner"/>

Commit message: Adjusted URDF model

File: wheelchair_description/urdf/wheelchair_description.xacro (robot description, xacro)
@@ -145,4 +145,5 @@
   </link>
 <!--Laser Scanners -->
+<!--Magic numbers for brute force turning-->
   <link name="right_scanner">
     <inertial>
@@ -153,5 +154,5 @@
   <joint name="right_scanner_joint" type="fixed">
     <axis xyz="0 0 0" />
-    <origin xyz="${chair_length/2 - 0.1/2 + chair_length/8} -${0.05/2 + .12} ${chair_height/16 + 0.05}" rpy="0 0 1.5707"/>
+    <origin xyz="${chair_length/2 - 0.1/2 + chair_length/8} -${0.05/2 + .1125} ${chair_height/16 + 0.05}" rpy="0 0 1.5707"/>
     <parent link="right_bar"/>
     <child link="right_scanner"/>
@@ -165,5 +166,5 @@
   <joint name="left_scanner_joint" type="fixed">
     <axis xyz="0 0 0" />
-    <origin xyz="${chair_length/2 - 0.1/2 + chair_length/8} ${0.05/2 + .12} ${chair_height/16 + 0.05}" rpy="0 0 -1.5707"/>
+    <origin xyz="${chair_length/2 - 0.1/2 + chair_length/8} ${0.05/2 + .1125} ${chair_height/16 + 0.05}" rpy="0 0 -1.5707"/>
     <parent link="left_bar"/>
     <child link="left_scanner"/>

Commit message: Modified URDF

File: wheelchair_description/urdf/wheelchair_description.xacro (robot description, xacro)
@@ -122,4 +122,9 @@
       </geometry>
     </collision>
+    <visual>
+      <geometry>
+        <cylinder length="${main_wheel_length}" radius="${main_wheel_radius}"/>
+      </geometry>
+    </visual>
     <inertial>
       <mass value="${main_wheel_weight}"/>
@@ -139,4 +144,9 @@
       </geometry>
     </collision>
+    <visual>
+      <geometry>
+        <cylinder length="${main_wheel_length}" radius="${main_wheel_radius}"/>
+      </geometry>
+    </visual>
     <inertial>
       <mass value="${main_wheel_weight}"/>
@@ -151,8 +161,14 @@
       <inertia ixx="1e-3" ixy="0" ixz="0" iyy="1e-3" iyz="0" izz="1e-3" />
     </inertial>
+    <visual>
+      <origin rpy="0 0 0" xyz="0 0 0"/>
+      <geometry>
+        <box size="0.05 0.05 0.05"/>
+      </geometry>
+    </visual>
   </link>
   <joint name="right_scanner_joint" type="fixed">
     <axis xyz="0 0 0" />
-    <origin xyz="${chair_length/2 - 0.1/2 + chair_length/8} -${0.05/2 + .1125} ${chair_height/16 + 0.05}" rpy="0 0 1.5707"/>
+    <origin xyz="${chair_length/2 - 0.1/2 + chair_length/8} -${0.05/2 + .1025} ${chair_height/16 + 0.05}" rpy="0 0 1.5707"/>
     <parent link="right_bar"/>
     <child link="right_scanner"/>
@@ -163,8 +179,14 @@
       <inertia ixx="1e-3" ixy="0" ixz="0" iyy="1e-3" iyz="0" izz="1e-3" />
     </inertial>
+    <visual>
+      <origin rpy="0 0 0" xyz="0 0 0"/>
+      <geometry>
+        <box size="0.05 0.05 0.05"/>
+      </geometry>
+    </visual>
   </link>
   <joint name="left_scanner_joint" type="fixed">
     <axis xyz="0 0 0" />
-    <origin xyz="${chair_length/2 - 0.1/2 + chair_length/8} ${0.05/2 + .1125} ${chair_height/16 + 0.05}" rpy="0 0 -1.5707"/>
+    <origin xyz="${chair_length/2 - 0.1/2 + chair_length/8} ${0.05/2 + .1025} ${chair_height/16 + 0.05}" rpy="0 0 -1.5707"/>
     <parent link="left_bar"/>
     <child link="left_scanner"/>
@@ -210,4 +232,9 @@
       </surface>
     </collision>
+    <visual>
+      <geometry>
+        <cylinder length="${small_wheel_length}" radius="${small_wheel_radius}"/>
+      </geometry>
+    </visual>
     <inertial>
       <mass value="${small_wheel_weight}"/>
@@ -254,4 +281,9 @@
       </surface>
     </collision>
+    <visual>
+      <geometry>
+        <cylinder length="${small_wheel_length}" radius="${small_wheel_radius}"/>
+      </geometry>
+    </visual>
     <inertial>
       <mass value="${small_wheel_weight}"/>
@@ -299,4 +331,9 @@
       </surface>
     </collision>
+    <visual>
+      <geometry>
+        <cylinder length="0.05" radius="${small_wheel_radius}"/>
+      </geometry>
+    </visual>
     <inertial>
       <mass value="${small_wheel_weight}"/>
@@ -343,4 +380,9 @@
       </surface>
     </collision>
+    <visual>
+      <geometry>
+        <cylinder length="0.05" radius="${small_wheel_radius}"/>
+      </geometry>
+    </visual>
     <inertial>
       <mass value="${small_wheel_weight}"/>

Commit message: Readjusted laser scanners in URDF

File: wheelchair_description/urdf/wheelchair_description.xacro (robot description, xacro)
@@ -170,5 +170,5 @@
   <joint name="right_scanner_joint" type="fixed">
     <axis xyz="0 0 0" />
-    <origin xyz="${chair_length/2 - 0.1/2 + chair_length/8} -${0.05/2 + .1025} ${chair_height/16 + 0.05}" rpy="0 0 1.5707"/>
+    <origin xyz="${chair_length/2 - 0.1/2 + chair_length/8} -${0.164} ${chair_height/16 + 0.05}" rpy="0 0 1.5707"/>
     <parent link="right_bar"/>
     <child link="right_scanner"/>
@@ -188,5 +188,5 @@
   <joint name="left_scanner_joint" type="fixed">
     <axis xyz="0 0 0" />
-    <origin xyz="${chair_length/2 - 0.1/2 + chair_length/8} ${0.05/2 + .1025} ${chair_height/16 + 0.05}" rpy="0 0 -1.5707"/>
+    <origin xyz="${chair_length/2 - 0.1/2 + chair_length/8} ${0.164} ${chair_height/16 + 0.05}" rpy="0 0 -1.5707"/>
     <parent link="left_bar"/>
     <child link="left_scanner"/>
