Commit message: Added new launch and bash files for full simulation launch
Files are "wheelchair_full_simulation.launch" in "wheelchair_bringup" and "gazebo_full_launch.bash" in "wheelchair_description"

Also fixed invisible chair in rviz issue (alpha settings in xacro files were wrong)

File: wheelchair_description/urdf/model.urdf (robot description, URDF)
Before this commit: robot wheelchair, 18 links, 17 joints
Joints:
- joint front_left_swivel_joint: origin xyz=-0.406 0.0 -0.148875 rpy=0 0 0 -> xyz=-0.446 -0.0725 -0.148875 rpy=0 0 0
- joint front_right_swivel_joint: origin xyz=-0.406 0.0 -0.148875 rpy=0 0 0 -> xyz=-0.446 0.0725 -0.148875 rpy=0 0 0
- joint left_bar_joint: origin xyz=0.0 -0.3215 -0.446625 rpy=0 0 0 -> xyz=0.0 -0.4215 -0.446625 rpy=0 0 0
- joint left_scanner_joint: origin xyz=0.4825 -0.025 0.1244375 rpy=0 0 -1.5707 -> xyz=0.4575 -0.0 0.1244375 rpy=0 0 -1.5707
- joint rear_left_swivel_joint: origin xyz=0.406 0.0 -0.148875 rpy=0 0 0 -> xyz=0.366 -0.035 -0.148875 rpy=0 0 0
- joint rear_right_swivel_joint: origin xyz=0.406 0.0 -0.148875 rpy=0 0 0 -> xyz=0.366 0.035 -0.148875 rpy=0 0 0
- joint right_bar_joint: origin xyz=0.0 0.3215 -0.446625 rpy=0 0 0 -> xyz=0.0 0.4215 -0.446625 rpy=0 0 0
- joint right_scanner_joint: origin xyz=0.4825 0.025 0.1244375 rpy=0 0 1.5707 -> xyz=0.4575 0.0 0.1244375 rpy=0 0 1.5707

File: wheelchair_description/urdf/wheelchair_description.xacro (robot description, xacro)
@@ -35,7 +35,7 @@
         <geometry>
     	    <mesh filename="package://wheelchair_description/meshes/Wheel_Chair.dae" scale="0.20 0.20 0.20"/>
-      </geometry>
+        </geometry>
       <material name="white">
-        <color rgba="1 1 0 .01"/>
+        <color rgba="1 1 0 1"/>
       </material>
     </visual>
@@ -94,5 +94,5 @@
     <parent link="base_link"/>
     <child link="right_bar"/>
-    <origin rpy="0 0 0" xyz="0.0 ${chair_width/2} -${chair_height/4 + chair_height/8}"/> <!--chair_height/4 + chair_height/8 because this is relative to the center of the bar -->
+    <origin rpy="0 0 0" xyz="0.0 ${chair_width/2 + .1} -${chair_height/4 + chair_height/8}"/> <!--chair_height/4 + chair_height/8 because this is relative to the center of the bar -->
   </joint>
 <!--Left Bar -->
@@ -107,5 +107,5 @@
     <parent link="base_link"/>
     <child link="left_bar"/>
-    <origin rpy="0 0 0" xyz="0.0 -${chair_width/2} -${chair_height/4 + chair_height/8}"/> <!--chair_height/4 + chair_height/8 because this is relative to the center of the bar -->
+    <origin rpy="0 0 0" xyz="0.0 -${chair_width/2 + .1} -${chair_height/4 + chair_height/8}"/> <!--chair_height/4 + chair_height/8 because this is relative to the center of the bar -->
   </joint>
 <!--Main Wheels -->
@@ -153,5 +153,5 @@
   <joint name="right_scanner_joint" type="fixed">
     <axis xyz="0 0 0" />
-    <origin xyz="${chair_length/2 - 0.05/2 + chair_length/8} ${0.05/2} ${chair_height/16 + 0.05}" rpy="0 0 1.5707"/>
+    <origin xyz="${chair_length/2 - 0.1/2 + chair_length/8} ${0.05/2 - .025} ${chair_height/16 + 0.05}" rpy="0 0 1.5707"/>
     <parent link="right_bar"/>
     <child link="right_scanner"/>
@@ -165,5 +165,5 @@
   <joint name="left_scanner_joint" type="fixed">
     <axis xyz="0 0 0" />
-    <origin xyz="${chair_length/2 - 0.05/2 + chair_length/8} -${0.05/2} ${chair_height/16 + 0.05}" rpy="0 0 -1.5707"/>
+    <origin xyz="${chair_length/2 - 0.1/2 + chair_length/8} -${0.05/2 - .025} ${chair_height/16 + 0.05}" rpy="0 0 -1.5707"/>
     <parent link="left_bar"/>
     <child link="left_scanner"/>
@@ -185,5 +185,5 @@
     <parent link="right_bar"/>
     <child link="front_right_swivel"/>
-    <origin rpy="0 0 0" xyz="-${chair_length/2} 0.0 -${chair_height/8}"/>
+    <origin rpy="0 0 0" xyz="-${chair_length/2 + .04} 0.0725 -${chair_height/8}"/>
     <dynamics damping="0.0" friction="0.5" />
   </joint>
@@ -229,5 +229,5 @@
     <parent link="left_bar"/>
     <child link="front_left_swivel"/>
-    <origin rpy="0 0 0" xyz="-${chair_length/2} 0.0 -${chair_height/8}"/>
+    <origin rpy="0 0 0" xyz="-${chair_length/2 + .04} -0.0725 -${chair_height/8}"/>
     <dynamics damping="0.0" friction="0.5" />
   </joint>
@@ -274,5 +274,5 @@
     <parent link="right_bar"/>
     <child link="rear_right_swivel"/>
-    <origin rpy="0 0 0" xyz="${chair_length/2} 0.0 -${chair_height/8}"/>
+    <origin rpy="0 0 0" xyz="${chair_length/2 - .04} 0.035 -${chair_height/8}"/>
     <dynamics damping="0.0" friction="0.5" />
   </joint>
@@ -314,9 +314,9 @@
     </inertial>
   </link>
-   <joint name="rear_left_swivel_joint" type="continuous">
+  <joint name="rear_left_swivel_joint" type="continuous">
     <axis xyz="0 0 1"/>
     <parent link="left_bar"/>
     <child link="rear_left_swivel"/>
-    <origin rpy="0 0 0" xyz="${chair_length/2} 0.0 -${chair_height/8}"/>
+    <origin rpy="0 0 0" xyz="${chair_length/2 - .04} -0.035 -${chair_height/8}"/>
     <dynamics damping="0.0" friction="0.5" />
   </joint>
@@ -358,13 +358,4 @@
       <visualize>true</visualize>
       <topic>__default_topic__</topic>
-      <plugin name="imu_plugin" filename="libgazebo_ros_imu_sensor.so">
-        <topicName>imu</topicName>
-        <bodyName>imu_link</bodyName>
-        <updateRateHZ>10.0</updateRateHZ>
-        <gaussianNoise>0.0</gaussianNoise>
-        <xyzOffset>0 0 0</xyzOffset>
-        <rpyOffset>0 0 0</rpyOffset>
-        <frameName>imu_link</frameName>
-      </plugin>
     </sensor>
   </gazebo>

Commit message: Changed test.world so the map origin is more useful for odometry
Spawning at (0, 0) will no longer cause issues. Gazebo uses only the map origin for simulated odometry, so spawning at (0, 0) is needed for accurate simulation.

File: wheelchair_description/urdf/model.urdf (robot description, URDF)
Before this commit: robot wheelchair, 18 links, 17 joints
Joints:
- joint base_footprint_joint: origin xyz= 0 0 .7 rpy=0 0 0 -> xyz= 0 0 0.7 rpy=0 0 0
- joint imu_joint: origin xyz=.32 0 -.35 rpy=3.14159265359 0 0 -> xyz=0.32 0 -0.35 rpy=3.14159265359 0 0

File: wheelchair_description/urdf/wheelchair_description.xacro (robot description, xacro)
@@ -16,4 +16,10 @@
   <xacro:property name="small_wheel_length" value=".05" />
   <xacro:property name="small_wheel_weight" value="1.0" />
+  <xacro:property name="imu_x" value=".32" />
+  <xacro:property name="imu_z" value="-.35" />
+  <xacro:property name="base_link_z" value="-.59" />
+  <xacro:property name="base_link_rot_y" value="-1.571" />
+  <xacro:property name="footprint_z" value=".1" />
+  <xacro:property name="footprint_joint_z" value=".7" />
   <xacro:macro name="box_intertia" params="height length width weight" >
     <inertia ixx="${1/12 * weight * (height + length)}" ixy="0" ixz="0" iyy="${1/12 * weight * (width + length)}" iyz="0" izz="${1/12 * weight * (width + height)}" />
@@ -23,8 +29,8 @@
   </xacro:macro>
   <link name="base_footprint">
-    <origin xyz="0 0 .1" rpy="0 0 0"/>
+    <origin xyz="0 0 ${footprint_z}" rpy="0 0 0"/>
   </link>
   <joint name="base_footprint_joint" type="fixed">
-    <origin xyz=" 0 0 .7" rpy="0 0 0"/>
+    <origin xyz=" 0 0 ${footprint_joint_z}" rpy="0 0 0"/>
     <parent link="base_footprint"/>
     <child link="base_link"/>
@@ -32,5 +38,5 @@
   <link name="base_link">
     <visual>
-      <origin xyz="0 0 -.59" rpy="0 0 -1.571" />
+      <origin xyz="0 0 ${base_link_z}" rpy="0 0 ${base_link_rot_y}" />
         <geometry>
     	    <mesh filename="package://wheelchair_description/meshes/Wheel_Chair.dae" scale="0.20 0.20 0.20"/>
@@ -41,5 +47,5 @@
     </visual>
     <collision>
-      <origin xyz="0 0 -.59" rpy="0 0 -1.571" />
+      <origin xyz="0 0 ${base_link_z}" rpy="0 0 ${base_link_rot_y}" />
       <geometry>
         <mesh filename="package://wheelchair_description/meshes/Wheel_Chair.dae" scale="0.20 0.20 0.20"/>
@@ -47,5 +53,5 @@
     </collision>
     <inertial>
-      <origin xyz="0 0 -.59" rpy="0 0 -1.571" />
+      <origin xyz="0 0 ${base_link_z}" rpy="0 0 ${base_link_rot_y}" />
       <mass value="${chair_weight}"/>
       <xacro:box_intertia height="${chair_height}" length="${chair_length}" width="${chair_width}" weight="${chair_weight}" />
@@ -68,5 +74,5 @@
     <parent link="base_link"/>
     <child link="imu_link"/>
-    <origin xyz=".32 0 -.35" rpy="${PI} 0 0"/>
+    <origin xyz="${imu_x} 0 ${imu_z}" rpy="${PI} 0 0"/>
   </joint>
 <!--Legs -->
@@ -355,6 +361,6 @@
     <plugin filename="libgazebo_ros_p3d.so" name="ground_truth">
       <always_on>true</always_on>
-      <frameName>map</frameName>
-      <bodyName>base_link</bodyName>
+      <frameName>world</frameName>
+      <bodyName>base_footprint</bodyName>
       <topicName>odom</topicName>
       <updateRate>30.0</updateRate>

Commit message: Added demo launch files and comments

File: wheelchair_description/urdf/model.urdf (robot description, URDF)
Before this commit: robot wheelchair, 18 links, 17 joints
Links:
- link front_left_wheel: geometry collision cylinder length=0.05 radius=0.089; visual cylinder length=0.05 radius=0.089
- link front_right_wheel: geometry collision cylinder length=0.05 radius=0.089; visual cylinder length=0.05 radius=0.089
- link left_main_wheel: geometry collision cylinder length=0.065 radius=0.165; visual cylinder length=0.065 radius=0.165
- link left_scanner: geometry visual box size=0.05 0.05 0.05
- link rear_left_wheel: geometry collision cylinder length=0.05 radius=0.089; visual cylinder length=0.05 radius=0.089
- link rear_right_wheel: geometry collision cylinder length=0.05 radius=0.089; visual cylinder length=0.05 radius=0.089
- link right_main_wheel: geometry collision cylinder length=0.065 radius=0.165; visual cylinder length=0.065 radius=0.165
- link right_scanner: geometry visual box size=0.05 0.05 0.05
Joints:
- joint left_scanner_joint: origin xyz=0.4575 -0.0 0.1244375 rpy=0 0 -1.5707 -> xyz=0.4575 0.1275 0.1244375 rpy=0 0 -1.5707
- joint right_scanner_joint: origin xyz=0.4575 0.0 0.1244375 rpy=0 0 1.5707 -> xyz=0.4575 -0.1275 0.1244375 rpy=0 0 1.5707

Commit message: Added test world for "move_to" demo. Added install and uninstall script prototypes

File: wheelchair_description/urdf/model.urdf (robot description, URDF)
Before this commit: robot wheelchair, 18 links, 17 joints
Joints:
- joint left_scanner_joint: origin xyz=0.4575 0.1275 0.1244375 rpy=0 0 -1.5707 -> xyz=0.4575 0.164 0.1244375 rpy=0 0 -1.5707
- joint right_scanner_joint: origin xyz=0.4575 -0.1275 0.1244375 rpy=0 0 1.5707 -> xyz=0.4575 -0.164 0.1244375 rpy=0 0 1.5707
